File: eagle/modules/nano/ethernet-v1/NanoRemotev2.brd (EAGLE design)
At the start: 113 x 82.5 mm, 59 parts, among them IC1 ULN2803A, IC2 ULN2803A, IC4 ULN2803A

Commit message: Update extension and create new nano I2C
Parts:
- removed A1: ANALOG1, lpatiny:RJ12-STRAIGHT-RS232
- removed A2: ANALOG2, lpatiny:RJ12-STRAIGHT-RS232
- removed RXTX_INT1: RS232, lpatiny:RJ12-STRAIGHT-RS232
Connections:
- net +12V: no longer A1.+12V, A2.+12V, RXTX_INT1.+12V
- net +5V: no longer A1.+5V, A2.+5V, RXTX_INT1.+5V
- net D2B5: no longer RXTX_INT1.TX
- net D2B8: no longer A1.TX
- net D2B9: no longer A2.TX
- net GND: no longer A1.GND1, A1.GND2, A1.RX, A2.GND1, A2.GND2, A2.RX, RXTX_INT1.GND1, RXTX_INT1.GND2
- net N$7: no longer RXTX_INT1.RX
Changed lines of the file:
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@@
 <element name="R2" library="resistor" package="M1206" value="1K" x="95.25" y="17.78" rot="R270"/>
 <element name="IC1" library="lpatiny" package="SO18W" value="ULN2803A" x="83.82" y="40.64" rot="MR0"/>
-<element name="RXTX_INT1" library="lpatiny" package="RJ12-STRAIGHT-RS232" value="RS232" x="104.14" y="46.99" rot="R90"/>
 <element name="R3" library="resistor" package="M1206" value="1K" x="90.17" y="54.61"/>
 <element name="D2_IO5" library="lpatiny" package="RJ12-STRAIGHT" value="IO5" x="80.01" y="74.93" rot="R180">
@@
 <element name="RL1" library="resistor" package="M1206" value="1K" x="90.17" y="60.96" rot="MR0"/>
 <element name="LED1" library="lpatiny" package="LED3MM" value="" x="96.52" y="59.69"/>
-<element name="A1" library="lpatiny" package="RJ12-STRAIGHT-RS232" value="ANALOG1" x="63.5" y="7.62"/>
 <element name="RA0" library="resistor" package="M1206" value="1K" x="67.31" y="22.86" rot="MR90"/>
-<element name="A2" library="lpatiny" package="RJ12-STRAIGHT-RS232" value="ANALOG2" x="80.01" y="7.62"/>
 <element name="RA1" library="resistor" package="M1206" value="1K" x="78.74" y="22.86" rot="MR270"/>
 <element name="RGB_5-6-11" library="lpatiny" package="LED-TRICOLOR-THROUGHHOLE" value="" x="30.7975" y="22.5425" rot="R270"/>
@@
 <contactref element="I2C_INT0" pad="GND1"/>
 <contactref element="I2C_INT0" pad="GND2"/>
-<contactref element="RXTX_INT1" pad="GND1"/>
-<contactref element="RXTX_INT1" pad="GND2"/>
 <contactref element="D2_IO5" pad="GND1"/>
 <contactref element="D2_IO5" pad="GND2"/>
 <contactref element="D3_IO6" pad="GND1"/>
 <contactref element="D3_IO6" pad="GND2"/>
-<contactref element="A1" pad="GND1"/>
-<contactref element="A1" pad="GND2"/>
-<contactref element="A2" pad="GND1"/>
-<contactref element="A2" pad="GND2"/>
 <contactref element="U$1" pad="GND2"/>
 <contactref element="U$1" pad="GND1"/>
-<contactref element="A1" pad="RX"/>
-<contactref element="A2" pad="RX"/>
 <contactref element="RA7" pad="2"/>
 <contactref element="RA6" pad="2"/>
@@
 <via x="83.185" y="30.48" extent="1-16" drill="0.6096"/>
 <via x="83.185" y="20.32" extent="1-16" drill="0.6096"/>
+<wire x1="97.79" y1="47.625" x2="97.79" y2="47.625" width="0" layer="19" extent="1-16"/>
 </signal>
 <signal name="+12V" class="2">
@@
 <contactref element="D12_IO4" pad="+12V"/>
 <contactref element="I2C_INT0" pad="+12V"/>
-<contactref element="RXTX_INT1" pad="+12V"/>
 <contactref element="D2_IO5" pad="+12V"/>
 <contactref element="D3_IO6" pad="+12V"/>
-<contactref element="A1" pad="+12V"/>
-<contactref element="A2" pad="+12V"/>
 <contactref element="U$1" pad="+12V"/>
 <contactref element="RL3" pad="2"/>
@@
 <via x="52.705" y="27.305" extent="1-16" drill="0.6096"/>
 <via x="52.705" y="17.78" extent="1-16" drill="0.6096"/>
+<wire x1="60.325" y1="16.51" x2="60.325" y2="16.51" width="0" layer="19" extent="1-16"/>
 </signal>
 <signal name="+5V" class="2">
@@
 <contactref element="RL12" pad="2"/>
 <contactref element="I2C_INT0" pad="+5V"/>
-<contactref element="RXTX_INT1" pad="+5V"/>
 <contactref element="D2_IO5" pad="+5V"/>
 <contactref element="RL0" pad="2"/>
 <contactref element="D3_IO6" pad="+5V"/>
 <contactref element="RL1" pad="2"/>
-<contactref element="A1" pad="+5V"/>
-<contactref element="A2" pad="+5V"/>
 <contactref element="U$1" pad="+5V"/>
 <contactref element="RL2" pad="2"/>
@@
 <via x="50.8" y="29.21" extent="1-16" drill="0.6096"/>
 <via x="65.405" y="29.21" extent="1-16" drill="0.6096"/>
+<wire x1="81.915" y1="16.51" x2="81.915" y2="16.51" width="0" layer="19" extent="1-16"/>
+<wire x1="65.405" y1="16.51" x2="65.405" y2="16.51" width="0" layer="19" extent="1-16"/>
 </signal>
 <signal name="3V3">
@@
 </signal>
 <signal name="D2B5">
-<contactref element="RXTX_INT1" pad="TX"/>
 <contactref element="R3" pad="1"/>
 <wire x1="88.265" y1="54.61" x2="86.995" y2="53.34" width="0.4572" layer="1"/>
@@
 </signal>
 <signal name="D2B8">
-<contactref element="A1" pad="TX"/>
 <contactref element="RA0" pad="1"/>
 <wire x1="62.865" y1="16.51" x2="67.31" y2="20.955" width="0.4572" layer="16"/>
@@
 </signal>
 <signal name="D2B9">
-<contactref element="A2" pad="TX"/>
 <contactref element="RA1" pad="1"/>
 <wire x1="80.01" y1="22.86" x2="78.74" y2="24.13" width="0.4572" layer="16"/>
@@
 <signal name="N$7">
 <contactref element="R1" pad="1"/>
-<contactref element="RXTX_INT1" pad="RX"/>
 <wire x1="88.9" y1="51.435" x2="90.805" y2="49.53" width="0.4572" layer="1"/>
 <wire x1="90.805" y1="49.53" x2="92.71" y2="49.53" width="0.4572" layer="1"/>
