File: eagle/modules/I2C/IO relay - external voltage/4channelsRelay.brd (EAGLE design)
At the start: 113 x 82.5 mm, 37 parts, among them IC2 MCP2300X/P, IC3 ULN2803, K1 JS-M1-9V-5, K2 JS-M1-9V-5, K3 JS-M1-9V-5, K4 JS-M1-9V-5, P1 WIREPAD3,81/1,4, P2 WIREPAD3,81/1,4, P3 WIREPAD3,81/1,4, P4 WIREPAD3,81/1,4

Commit message: New relay version for switch
Parts:
- added P5, P6, P7, P8: WIREPAD3,81/1,4, wirepad:3,81/1,4
- moved PC4 1.27 mm to (74.9, 64.8)
- moved P2 1.27 mm to (45.1, 64.8)
- moved P3 1.27 mm to (62.9, 64.8)
- moved P1 1.27 mm to (27.3, 64.8)
- moved PC1 1.27 mm to (21.6, 64.8)
- moved P4 1.27 mm to (80.6, 64.8)
- moved PC2 1.27 mm to (39.4, 64.8)
- moved PC3 1.27 mm to (57.1, 64.8)
Connections:
- new net N$10: K3.NC, P6.1
- new net N$13: K4.NC, P5.1
- new net N$6: K1.NC, P8.1
- new net N$7: K2.NC, P7.1
Routing:
- net N$7: track 0.00 -> 11.3 mm
- net N$10: track 0.00 -> 11.3 mm
- net N$13: track 0.00 -> 11.3 mm
- net N$6: track 0.00 -> 11.0 mm
- net N$14: track 12.6 -> 11.3 mm
- net N$11: track 12.6 -> 11.3 mm
- net N$19: track 12.6 -> 11.3 mm
- net N$8: track 12.6 -> 11.3 mm
- net N$12: track 100.3 -> 99.1 mm
Changed lines of the file:
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@@
 <setting verticaltext="up"/>
 </settings>
-<grid distance="0.05" unitdist="inch" unit="mm" style="lines" multiple="1" display="no" altdistance="0.025" altunitdist="inch" altunit="inch"/>
+<grid distance="0.05" unitdist="inch" unit="inch" style="lines" multiple="1" display="no" altdistance="0.025" altunitdist="inch" altunit="inch"/>
 <layers>
 <layer number="1" name="Top" color="4" fill="1" visible="yes" active="yes"/>
@@
 <attribute name="OC_NEWARK" value="unknown" x="74.93" y="48.26" size="1.778" layer="27" rot="R270" display="off"/>
 </element>
-<element name="PC1" library="wirepad" package="3,81/1,4" value="WIREPAD3,81/1,4" x="20.32" y="64.77"/>
-<element name="PC2" library="wirepad" package="3,81/1,4" value="WIREPAD3,81/1,4" x="38.1" y="64.77"/>
-<element name="P2" library="wirepad" package="3,81/1,4" value="WIREPAD3,81/1,4" x="43.815" y="64.77"/>
-<element name="P1" library="wirepad" package="3,81/1,4" value="WIREPAD3,81/1,4" x="26.035" y="64.77"/>
-<element name="P3" library="wirepad" package="3,81/1,4" value="WIREPAD3,81/1,4" x="61.595" y="64.77"/>
-<element name="PC3" library="wirepad" package="3,81/1,4" value="WIREPAD3,81/1,4" x="55.88" y="64.77"/>
-<element name="PC4" library="wirepad" package="3,81/1,4" value="WIREPAD3,81/1,4" x="73.66" y="64.77"/>
-<element name="P4" library="wirepad" package="3,81/1,4" value="WIREPAD3,81/1,4" x="79.375" y="64.77"/>
+<element name="PC1" library="wirepad" package="3,81/1,4" value="WIREPAD3,81/1,4" x="21.59" y="64.77"/>
+<element name="PC2" library="wirepad" package="3,81/1,4" value="WIREPAD3,81/1,4" x="39.37" y="64.77"/>
+<element name="P2" library="wirepad" package="3,81/1,4" value="WIREPAD3,81/1,4" x="45.085" y="64.77"/>
+<element name="P1" library="wirepad" package="3,81/1,4" value="WIREPAD3,81/1,4" x="27.305" y="64.77"/>
+<element name="P3" library="wirepad" package="3,81/1,4" value="WIREPAD3,81/1,4" x="62.865" y="64.77"/>
+<element name="PC3" library="wirepad" package="3,81/1,4" value="WIREPAD3,81/1,4" x="57.15" y="64.77"/>
+<element name="PC4" library="wirepad" package="3,81/1,4" value="WIREPAD3,81/1,4" x="74.93" y="64.77"/>
+<element name="P4" library="wirepad" package="3,81/1,4" value="WIREPAD3,81/1,4" x="80.645" y="64.77"/>
 <element name="POWER2" library="wirepad" package="3,81/1,4" value="WIREPAD3,81/1,4" x="95.25" y="64.77"/>
 <element name="PAD10" library="wirepad" package="3,81/1,4" value="WIREPAD3,81/1,4" x="95.25" y="57.15"/>
 <element name="IC2" library="adafruit" package="DIL18" value="MCP2300X/P" x="36.83" y="13.97"/>
+<element name="P5" library="wirepad" package="3,81/1,4" value="WIREPAD3,81/1,4" x="69.215" y="64.77"/>
+<element name="P6" library="wirepad" package="3,81/1,4" value="WIREPAD3,81/1,4" x="51.435" y="64.77"/>
+<element name="P7" library="wirepad" package="3,81/1,4" value="WIREPAD3,81/1,4" x="33.655" y="64.77"/>
+<element name="P8" library="wirepad" package="3,81/1,4" value="WIREPAD3,81/1,4" x="15.875" y="64.77"/>
 </elements>
 <signals>
@@
 <contactref element="P4" pad="1"/>
 <contactref element="K4" pad="NO"/>
-<wire x1="79.375" y1="64.77" x2="80.93" y2="64.77" width="2.1844" layer="16"/>
+<wire x1="80.645" y1="64.77" x2="80.93" y2="64.77" width="2.1844" layer="16"/>
 <wire x1="80.93" y1="64.77" x2="80.93" y2="53.76" width="2.1844" layer="16"/>
 </signal>
@@
 <contactref element="P3" pad="1"/>
 <contactref element="K3" pad="NO"/>
-<wire x1="61.595" y1="64.77" x2="63.15" y2="64.77" width="2.1844" layer="16"/>
+<wire x1="62.865" y1="64.77" x2="63.15" y2="64.77" width="2.1844" layer="16"/>
 <wire x1="63.15" y1="64.77" x2="63.15" y2="53.76" width="2.1844" layer="16"/>
 </signal>
@@
 <contactref element="P2" pad="1"/>
 <contactref element="K2" pad="NO"/>
-<wire x1="43.815" y1="64.77" x2="45.37" y2="64.77" width="2.1844" layer="16"/>
+<wire x1="45.085" y1="64.77" x2="45.37" y2="64.77" width="2.1844" layer="16"/>
 <wire x1="45.37" y1="64.77" x2="45.37" y2="53.76" width="2.1844" layer="16"/>
 </signal>
@@
 <contactref element="P1" pad="1"/>
 <contactref element="K1" pad="NO"/>
-<wire x1="26.035" y1="64.77" x2="27.59" y2="64.77" width="2.1844" layer="16"/>
+<wire x1="27.305" y1="64.77" x2="27.59" y2="64.77" width="2.1844" layer="16"/>
 <wire x1="27.59" y1="64.77" x2="27.59" y2="53.76" width="2.1844" layer="16"/>
 </signal>
@@
 <contactref element="PC1" pad="1"/>
 <wire x1="95.25" y1="64.77" x2="95.25" y2="69.85" width="2.1844" layer="16"/>
-<wire x1="95.25" y1="69.85" x2="73.66" y2="69.85" width="2.1844" layer="16"/>
-<wire x1="73.66" y1="64.77" x2="73.66" y2="69.85" width="2.1844" layer="16"/>
-<wire x1="73.66" y1="69.85" x2="55.88" y2="69.85" width="2.1844" layer="16"/>
-<wire x1="55.88" y1="64.77" x2="55.88" y2="69.85" width="2.1844" layer="16"/>
-<wire x1="55.88" y1="69.85" x2="38.1" y2="69.85" width="2.1844" layer="16"/>
-<wire x1="38.1" y1="64.77" x2="38.1" y2="69.85" width="2.1844" layer="16"/>
-<wire x1="38.1" y1="69.85" x2="20.32" y2="69.85" width="2.1844" layer="16"/>
-<wire x1="20.32" y1="69.85" x2="20.32" y2="64.77" width="2.1844" layer="16"/>
+<wire x1="95.25" y1="69.85" x2="74.93" y2="69.85" width="2.1844" layer="16"/>
+<wire x1="74.93" y1="64.77" x2="74.93" y2="69.85" width="2.1844" layer="16"/>
+<wire x1="74.93" y1="69.85" x2="57.15" y2="69.85" width="2.1844" layer="16"/>
+<wire x1="57.15" y1="64.77" x2="57.15" y2="69.85" width="2.1844" layer="16"/>
+<wire x1="57.15" y1="69.85" x2="39.37" y2="69.85" width="2.1844" layer="16"/>
+<wire x1="39.37" y1="64.77" x2="39.37" y2="69.85" width="2.1844" layer="16"/>
+<wire x1="39.37" y1="69.85" x2="21.59" y2="69.85" width="2.1844" layer="16"/>
+<wire x1="21.59" y1="69.85" x2="21.59" y2="64.77" width="2.1844" layer="16"/>
+</signal>
+<signal name="N$6" class="2">
+<contactref element="K1" pad="NC"/>
+<contactref element="P8" pad="1"/>
+<wire x1="15.59" y1="53.76" x2="15.875" y2="55.665" width="2.1844" layer="16"/>
+<wire x1="15.875" y1="55.665" x2="15.875" y2="64.77" width="2.1844" layer="16"/>
+</signal>
+<signal name="N$7" class="2">
+<contactref element="P7" pad="1"/>
+<contactref element="K2" pad="NC"/>
+<wire x1="33.37" y1="53.76" x2="33.655" y2="53.76" width="2.1844" layer="16"/>
+<wire x1="33.655" y1="53.76" x2="33.655" y2="64.77" width="2.1844" layer="16"/>
+</signal>
+<signal name="N$10" class="2">
+<contactref element="K3" pad="NC"/>
+<contactref element="P6" pad="1"/>
+<wire x1="51.15" y1="53.76" x2="51.435" y2="53.76" width="2.1844" layer="16"/>
+<wire x1="51.435" y1="53.76" x2="51.435" y2="64.77" width="2.1844" layer="16"/>
+</signal>
+<signal name="N$13" class="2">
+<contactref element="P5" pad="1"/>
+<contactref element="K4" pad="NC"/>
+<wire x1="68.93" y1="53.76" x2="69.215" y2="53.76" width="2.1844" layer="16"/>
+<wire x1="69.215" y1="53.76" x2="69.215" y2="64.77" width="2.1844" layer="16"/>
 </signal>
 </signals>
