File: eagle/modules/I2C/IO relay - external voltage/4channelsRelay.sch (EAGLE design)
At the start: 37 parts, among them IC2 MCP2300X/P, IC3 ULN2803, K1 JS-M1-9V-5, K2 JS-M1-9V-5, K3 JS-M1-9V-5, K4 JS-M1-9V-5, P1 WIREPAD3,81/1,4, P2 WIREPAD3,81/1,4, P3 WIREPAD3,81/1,4, P4 WIREPAD3,81/1,4

Commit message: New relay version for switch
Parts:
- added P5, P6, P7, P8: WIREPAD3,81/1,4, wirepad:WIREPAD3,81/1,4
Connections:
- new net N$10: K32.O, P6.P
- new net N$13: K42.O, P5.P
- new net N$6: K12.O, P8.P
- new net N$7: K22.O, P7.P
Changed lines of the file:
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@@
 <part name="IC2" library="adafruit" deviceset="MCP2300X" device="/P"/>
 <part name="P+6" library="supply1" deviceset="+5V" device=""/>
+<part name="P5" library="wirepad" deviceset="WIREPAD" device="3,81/1,4"/>
+<part name="P6" library="wirepad" deviceset="WIREPAD" device="3,81/1,4"/>
+<part name="P7" library="wirepad" deviceset="WIREPAD" device="3,81/1,4"/>
+<part name="P8" library="wirepad" deviceset="WIREPAD" device="3,81/1,4"/>
 </parts>
 <sheets>
@@
 <attribute name="VALUE" x="114.935" y="126.365" size="1.27" layer="96"/>
 </instance>
+<instance part="P5" gate="G$1" x="261.62" y="114.3" rot="R180"/>
+<instance part="P6" gate="G$1" x="261.62" y="137.16" rot="R180"/>
+<instance part="P7" gate="G$1" x="261.62" y="160.02" rot="R180"/>
+<instance part="P8" gate="G$1" x="261.62" y="182.88" rot="R180"/>
 </instances>
 <busses>
@@
 </segment>
 </net>
+<net name="N$6" class="2">
+<segment>
+<pinref part="K1" gate="2" pin="O"/>
+<pinref part="P8" gate="G$1" pin="P"/>
+<wire x1="241.3" y1="182.88" x2="259.08" y2="182.88" width="0.1524" layer="91"/>
+</segment>
+</net>
+<net name="N$7" class="2">
+<segment>
+<pinref part="P7" gate="G$1" pin="P"/>
+<pinref part="K2" gate="2" pin="O"/>
+<wire x1="259.08" y1="160.02" x2="241.3" y2="160.02" width="0.1524" layer="91"/>
+</segment>
+</net>
+<net name="N$10" class="2">
+<segment>
+<pinref part="K3" gate="2" pin="O"/>
+<pinref part="P6" gate="G$1" pin="P"/>
+<wire x1="241.3" y1="137.16" x2="259.08" y2="137.16" width="0.1524" layer="91"/>
+</segment>
+</net>
+<net name="N$13" class="2">
+<segment>
+<pinref part="P5" gate="G$1" pin="P"/>
+<pinref part="K4" gate="2" pin="O"/>
+<wire x1="259.08" y1="114.3" x2="241.3" y2="114.3" width="0.1524" layer="91"/>
+</segment>
+</net>
