File: eagle/modules/I2C/IO relay - external voltage/v2/4channelsRelayv2.brd (EAGLE design)
At the start: 100.3 x 74.9 mm, 41 parts, among them IC2 MCP2300X/P, IC3 ULN2803, K1 JS-M1-9V-5, K2 JS-M1-9V-5, K3 JS-M1-9V-5, K4 JS-M1-9V-5, P1 WIREPAD3,81/1,4, P2 WIREPAD3,81/1,4, P3 WIREPAD3,81/1,4, P4 WIREPAD3,81/1,4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

Commit message: Correct bug with pin 6 to 5V
Connections:
- net +5V: now also IC2.6
Routing:
- net +5V: track 277.7 -> 284.1 mm
Changed lines of the file:
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@@
 <wire x1="59.69" y1="16.51" x2="59.82" y2="16.51" width="1.3716" layer="16"/>
 <wire x1="41.91" y1="6.35" x2="43.18" y2="5.08" width="1.3716" layer="1"/>
-<wire x1="41.91" y1="21.59" x2="41.91" y2="7.62" width="1.3716" layer="1"/>
+<wire x1="41.91" y1="21.59" x2="41.91" y2="17.78" width="1.3716" layer="1"/>
+<wire x1="41.91" y1="17.78" x2="41.91" y2="7.62" width="1.3716" layer="1"/>
 <wire x1="41.91" y1="7.62" x2="41.91" y2="6.35" width="1.3716" layer="1"/>
 <wire x1="44.45" y1="24.13" x2="41.91" y2="21.59" width="1.3716" layer="1"/>
@@
 <wire x1="41.91" y1="7.62" x2="36.83" y2="2.54" width="1.3716" layer="1"/>
 <via x="36.83" y="2.54" extent="1-16" drill="0.6096"/>
+<contactref element="IC2" pad="6"/>
+<wire x1="41.91" y1="17.78" x2="35.56" y2="17.78" width="1.3716" layer="1"/>
 </signal>
 <signal name="N$38">

Commit message: update RESET pin to put a resistor of 10k to +5V
Parts:
- added R1: 10k, resistor:M1206
- R13, R14: value reserve -> 10k
Connections:
- new net N$15: IC2.6, R1.1
- net +5V: now also R1.2; no longer IC2.6
Routing:
- net GND: track 172.1 -> 119.0 mm
- net N$9: track 117.0 -> 84.8 mm, vias 1 -> 3
- net N$15: track 0.00 -> 28.4 mm
- net N$1: track 64.9 -> 84.5 mm, vias 0 -> 2
- net P1: track 30.3 -> 45.4 mm
- net SCL: track 72.0 -> 85.7 mm
- net N$18: track 14.5 -> 27.9 mm
- net N$16: track 23.0 -> 34.6 mm
- net P0: track 25.1 -> 36.4 mm
- net N$40: track 70.0 -> 80.6 mm, vias 2 -> 0
- net SDA: track 92.9 -> 101.3 mm, vias 0 -> 1
- net N$17: track 25.0 -> 17.0 mm
- net N$5: track 27.2 -> 20.8 mm
- net +5V: track 284.1 -> 286.2 mm, vias 1 -> 3
- net N$4: track 5.08 -> 7.01 mm
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