File: eagle/modules/pico/v1/v1.sch (EAGLE design)
At the start: 36 parts, among them IC1 MEGA8-AI, IC3 ULN2803A, IC4 ULN2803A, J1 RJ12STRAIGHT-RS232-SERVER

Commit message: Update pico
Parts:
- added C3: 10uF 20V, SparkFun:CAP_POL1206-KIT
- added C4: 100 nF, SparkFun:CAP1206
- added D1: 1N581D1206, lpatiny:1N581D1206
- added LED4: LED3MM, lpatiny:LED3MM
- added Q1: FDN340P, lpatiny:FDN360P
- added RL4: 1K, resistor:R-EU_M1206
Connections:
- new net 5V: C1.1, C2.1, C3.+, C4.1, D1.C, IC1.AVCC, IC1.VCC@1, IC1.VCC@2, Q1.S, R1.2, R7.2, R8.2, RL4.1, U$1.VCC
- new net ISP+5V: CON1.VCC, D1.A, Q1.G
- new net N$7: LED4.A, RL4.2
- net +5V: now also Q1.D; no longer C1.1, C2.1, CON1.VCC, IC1.AVCC, IC1.VCC@1, IC1.VCC@2, R1.2, R7.2, R8.2, U$1.VCC
- net GND: now also C3.-, C4.2, LED4.C
Other:
- moved on the sheet: CON1

Commit message: Update board size
Connections:
- removed net D13: LED1.A
- net SCK: now also LED1.A
Changed lines of the file:
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@@
 <label x="86.36" y="10.16" size="1.27" layer="95"/>
+</segment>
+<segment>
+<pinref part="LED1" gate="G$1" pin="A"/>
+<wire x1="-71.12" y1="101.6" x2="-73.66" y2="101.6" width="0.1524" layer="91"/>
+<label x="-75.184" y="102.362" size="1.27" layer="95"/>
 </segment>
 </net>
@@
 </segment>
 </net>
-<net name="D13" class="0">
-<segment>
-<pinref part="LED1" gate="G$1" pin="A"/>
-<wire x1="-71.12" y1="101.6" x2="-73.66" y2="101.6" width="0.1524" layer="91"/>
-<label x="-75.184" y="102.362" size="1.27" layer="95"/>
-</segment>
-</net>

Commit message: Remove transistor
Parts:
- removed C4: 100 nF, SparkFun:CAP1206
- removed Q1: FDN340P, lpatiny:FDN360P
- added D2: 1N581D1206, lpatiny:1N581D1206
Connections:
- net +5V: now also D2.A; no longer Q1.D
- net 5V: now also D2.C; no longer C4.1, Q1.S
- net GND: no longer C4.2
- net ISP+5V: no longer Q1.G
Changed lines of the file:
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@@
 <part name="U$6" library="SparkFun" deviceset="5V" device=""/>
 <part name="C3" library="SparkFun" deviceset="CAP_POL" device="1206-KIT" value="10uF 20V"/>
-<part name="C4" library="SparkFun" deviceset="CAP" device="1206" value="100 nF"/>
 <part name="D1" library="lpatiny" deviceset="1N581*" device="D1206" value="1N581D1206"/>
 <part name="GND3" library="supply1" deviceset="GND" device=""/>
@@
 <part name="RL4" library="resistor" deviceset="R-EU_" device="M1206" value="1K"/>
 <part name="P+1" library="supply1" deviceset="+5V" device=""/>
-<part name="Q1" library="lpatiny" deviceset="FDN360P" device="" value="FDN340P"/>
+<part name="D2" library="lpatiny" deviceset="1N581*" device="D1206" value="1N581D1206"/>
 </parts>
 <sheets>
@@
 <instance part="U$6" gate="G$1" x="20.32" y="30.48"/>
 <instance part="C3" gate="G$1" x="55.88" y="132.08"/>
-<instance part="C4" gate="G$1" x="63.5" y="129.54"/>
 <instance part="D1" gate="G$1" x="35.56" y="147.32"/>
 <instance part="GND3" gate="1" x="50.8" y="124.46"/>
@@
 <attribute name="VALUE" x="17.145" y="137.795" size="1.27" layer="96" rot="R180"/>
 </instance>
-<instance part="Q1" gate="G$1" x="27.94" y="137.16" rot="R270"/>
+<instance part="D2" gate="G$1" x="27.94" y="134.62"/>
 </instances>
 <busses>
@@
 <segment>
 <pinref part="C3" gate="G$1" pin="-"/>
-<pinref part="C4" gate="G$1" pin="2"/>
-<wire x1="55.88" y1="127" x2="63.5" y2="127" width="0.1524" layer="91"/>
 <pinref part="GND3" gate="1" pin="GND"/>
 <wire x1="50.8" y1="127" x2="55.88" y2="127" width="0.1524" layer="91"/>
-<junction x="63.5" y="127"/>
 <junction x="55.88" y="127"/>
 <junction x="50.8" y="127"/>
 <pinref part="LED4" gate="G$1" pin="C"/>
-<wire x1="81.28" y1="127" x2="63.5" y2="127" width="0.1524" layer="91"/>
+<wire x1="81.28" y1="127" x2="55.88" y2="127" width="0.1524" layer="91"/>
 </segment>
 </net>
@@
 <net name="5V" class="1">
 <segment>
-<wire x1="33.02" y1="134.62" x2="43.18" y2="134.62" width="0.1524" layer="91"/>
+<wire x1="30.48" y1="134.62" x2="43.18" y2="134.62" width="0.1524" layer="91"/>
 <label x="33.02" y="134.62" size="1.778" layer="95"/>
 <pinref part="U$3" gate="G$1" pin="5V"/>
@@
 <wire x1="43.18" y1="147.32" x2="43.18" y2="134.62" width="0.1524" layer="91"/>
 <pinref part="C3" gate="G$1" pin="+"/>
-<pinref part="C4" gate="G$1" pin="1"/>
-<wire x1="55.88" y1="134.62" x2="63.5" y2="134.62" width="0.1524" layer="91"/>
+<wire x1="55.88" y1="134.62" x2="68.58" y2="134.62" width="0.1524" layer="91"/>
 <wire x1="50.8" y1="134.62" x2="55.88" y2="134.62" width="0.1524" layer="91"/>
 <junction x="43.18" y="134.62"/>
 <junction x="50.8" y="134.62"/>
 <junction x="55.88" y="134.62"/>
-<junction x="63.5" y="134.62"/>
 <pinref part="RL4" gate="G$1" pin="1"/>
-<wire x1="63.5" y1="134.62" x2="68.58" y2="134.62" width="0.1524" layer="91"/>
-<pinref part="Q1" gate="G$1" pin="S"/>
-<junction x="33.02" y="134.62"/>
+<pinref part="D2" gate="G$1" pin="C"/>
 </segment>
 <segment>
@@
 <segment>
 <pinref part="P+1" gate="1" pin="+5V"/>
-<pinref part="Q1" gate="G$1" pin="D"/>
-<wire x1="17.78" y1="134.62" x2="22.86" y2="134.62" width="0.1524" layer="91"/>
+<wire x1="17.78" y1="134.62" x2="25.4" y2="134.62" width="0.1524" layer="91"/>
+<pinref part="D2" gate="G$1" pin="A"/>
 </segment>
 <segment>
@@
 <segment>
 <pinref part="CON1" gate="G$1" pin="VCC"/>
-<wire x1="2.54" y1="147.32" x2="30.48" y2="147.32" width="0.1524" layer="91"/>
+<wire x1="2.54" y1="147.32" x2="33.02" y2="147.32" width="0.1524" layer="91"/>
 <label x="5.08" y="149.86" size="1.778" layer="95"/>
-<wire x1="30.48" y1="139.7" x2="30.48" y2="147.32" width="0.1524" layer="91"/>
 <pinref part="D1" gate="G$1" pin="A"/>
-<wire x1="30.48" y1="147.32" x2="33.02" y2="147.32" width="0.1524" layer="91"/>
-<junction x="30.48" y="147.32"/>
-<pinref part="Q1" gate="G$1" pin="G"/>
-<junction x="30.48" y="139.7"/>
-</segment>
-</net>
+</segment>
+</net>

Commit message: Arduino ethernet first version
Parts:
- removed J2: (no value), tag-connect:TC2030-MCP
- added CON2: (no value), lpatiny:TINYISPTAG
Connections:
- removed net N$10: J2.ICSP_CLK/PGC
- removed net N$100: J2.VPP/MCLR
- removed net N$101: J2.VDD
- removed net N$102: J2.VSS(GND)
- removed net N$11: J2.LVP
- removed net N$9: J2.ICSP_DAT/PGD
- net +5V: now also U$1.VCC
- net 5V: no longer U$1.VCC
- net GND: now also CON2.GND
- net ISP+5V: now also CON2.VCC
- net MISO: now also CON2.MISO
- net MOSI: now also CON2.MOSI
- net RESET: now also CON2.RESET
- net SCK: now also CON2.SCK
