File: eagle/modules/stepper/stepper-v1.sch (EAGLE design)
At the start: 11 parts, among them J1 RJ12RIGHTANGLE

Commit message: Update Stepper
Parts:
- removed R3, R4: 1k, SparkFun:RESISTOR1206
- removed T1, T2: (no value), transistor:MMBT2222ALT1-NPN-SOT23-BEC
- added IC2: SN74LVC2G14, lpatiny:SN74LVC2G14
- added U$1, U$2, U$3, U$4: LED3MM, lpatiny:LED3MM
- added X1: (no value), con-wago-500:W237-6
Connections:
- removed net N$15: IC1.I7, IC1.I8, R4.2, T2.C
- new net N$10: R2.1, U$2.C
- new net N$11: R6.1, U$3.C
- new net N$12: R7.1, U$4.C
- new net N$7: IC1.I7, IC1.I8, IC2B.O
- new net N$9: R1.1, U$1.C
- net +12V: now also X1-2.KL, X1-5.KL
- net +5V: now also IC2P.VCC, U$1.A, U$2.A, U$3.A, U$4.A; no longer R3.1, R4.1
- net GND: now also IC2P.GND; no longer T1.E, T2.E
- net N$1: now also IC2A.I; no longer T1.B
- net N$14: now also IC1.I5, IC1.I6, IC2A.O; no longer IC1.I3, IC1.I4, R3.2, T1.C
- net N$2: now also IC1.I3, IC1.I4, IC2B.I; no longer IC1.I5, IC1.I6, T2.B
- net N$3: now also X1-6.KL
- net N$4: now also X1-4.KL
- net N$5: now also X1-3.KL
- net N$6: now also X1-1.KL
