File: eagle/modules/femto/v1.1-unrouted/femto.brd (EAGLE design)
At the start: 50.2 x 25.1 mm, 29 parts, among them IC1 MEGA8-AI, J1 RJ12RIGHTANGLE-I2C, J2 RJ12RIGHTANGLE-I2C

Commit message: femto routing
Parts:
- removed DB1, DB2, DC1, DC4: (no value), led:LED3MM
- added LED4, LED5, LED6: LED3MM, lpatiny:LED3MM
- added LED7: (no value), adafruit:CHIP-LED0603
- LED3: value (none) -> LED3MM; device adafruit:CHIP-LED0603 -> lpatiny:LED3MM
- moved LED3 14.7 mm to (32.4, 17.8), turned to 90 degrees
- moved LED1 7.62 mm to (18.4, 19.1)
- moved LED2 7.62 mm to (26.0, 19.1)
- renumbered R1 to R8, R2 to R7, RB1 to R5, RB2 to R4, RC1 to R3, RC6 to R6, RD10 to R2C, RD11 to R1A, RD12 to R1B, RD13 to R1C, RD8 to R2A, RD9 to R2B
Connections:
- net GND: now also LED3.K, LED4.K, LED5.K, LED6.K, LED7.C; no longer DB1.K, DB2.K, DC1.K, DC4.K, LED3.C
- net N$1: now also LED2.RED; no longer LED1.RED
- net N$15: now also LED7.A; no longer LED3.A
- net N$16: now also LED3.A; no longer DC1.A
- net N$20: now also LED1.RED; no longer LED2.RED
- net N$21: now also LED1.BLU; no longer LED2.BLU
- net N$22: now also LED1.GRN; no longer LED2.GRN
- net N$23: now also LED6.A; no longer DC4.A
- net N$40: now also LED5.A; no longer DB1.A
- net N$41: now also LED4.A; no longer DB2.A
- net N$7: now also LED2.BLU; no longer LED1.BLU
- net N$8: now also LED2.GRN; no longer LED1.GRN
