File: eagle/modules/femto/v1.1-unrouted/femto.sch (EAGLE design)
At the start: 29 parts, among them IC1 MEGA8-AI, J1 RJ12RIGHTANGLE-I2C, J2 RJ12RIGHTANGLE-I2C

Commit message: femto routing
Parts:
- removed DB1, DB2, DC1, DC4: (no value), led:LED3MM
- added LED4, LED5, LED6: LED3MM, lpatiny:LED3MM
- added LED7: (no value), adafruit:LEDCHIP-LED0603
- LED3: value (none) -> LED3MM; device adafruit:LEDCHIP-LED0603 -> lpatiny:LED3MM
- renumbered R1 to R8, R2 to R7, RB1 to R5, RB2 to R4, RC1 to R3, RC6 to R6, RD10 to R2C, RD11 to R1A, RD12 to R1B, RD13 to R1C, RD8 to R2A, RD9 to R2B
Connections:
- net GND: now also LED4.C, LED5.C, LED6.C, LED7.C; no longer DB1.C, DB2.C, DC1.C, DC4.C
- net N$1: now also LED2.CRED; no longer LED1.CRED
- net N$15: now also LED7.A; no longer LED3.A
- net N$16: now also LED3.A; no longer DC1.A
- net N$20: now also LED1.CRED; no longer LED2.CRED
- net N$21: now also LED1.CBLUE; no longer LED2.CBLUE
- net N$22: now also LED1.CGREEN; no longer LED2.CGREEN
- net N$23: now also LED6.A; no longer DC4.A
- net N$40: now also LED5.A; no longer DB1.A
- net N$41: now also LED4.A; no longer DB2.A
- net N$7: now also LED2.CBLUE; no longer LED1.CBLUE
- net N$8: now also LED2.CGREEN; no longer LED1.CGREEN
Other:
- moved on the sheet: LED1, LED2, LED3
