File: eagle/modules/I2C/LCD-MCP23008/v1.1/lcd-i2c.brd (EAGLE design)
At the start: 49.5 x 39.4 mm, 18 parts, among them IC1 MCP2300X/P, J2 RJ12RIGHTANGLE-I2C, J3 RJ12RIGHTANGLE-I2C, Q1 BC349

Commit message: Update file and library
Parts:
- R4, R5: value 10k -> UNUSED
Changed lines of the file:
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@@
 <element name="R1" library="adafruit" package="M1206" value="10k" x="24.13" y="35.56" smashed="yes">
 <attribute name="NAME" x="22.098" y="34.417" size="1.016" layer="25" font="vector" rot="R90"/>
-<attribute name="VALUE" x="20.193" y="36.195" size="1.27" layer="27" rot="R180"/>
+<attribute name="VALUE" x="24.638" y="38.1" size="1.27" layer="27" rot="R180"/>
 </element>
 <element name="R2" library="adafruit" package="M1206" value="10k" x="17.78" y="35.56" smashed="yes">
 <attribute name="NAME" x="15.748" y="34.417" size="1.016" layer="25" font="vector" rot="R90"/>
-<attribute name="VALUE" x="13.843" y="36.068" size="1.27" layer="27" rot="R180"/>
+<attribute name="VALUE" x="18.288" y="37.973" size="1.27" layer="27" rot="R180"/>
 </element>
 <element name="R3" library="adafruit" package="M1206" value="10k" x="11.43" y="35.687" smashed="yes">
 <attribute name="NAME" x="9.398" y="34.671" size="1.016" layer="25" font="vector" rot="R90"/>
-<attribute name="VALUE" x="7.62" y="36.449" size="1.27" layer="27" rot="R180"/>
+<attribute name="VALUE" x="12.065" y="38.354" size="1.27" layer="27" rot="R180"/>
 </element>
 <element name="A2" library="jumper" package="SJ" value="" x="10.16" y="29.21" smashed="yes" rot="R270">
@@
 <attribute name="VALUE" x="3.81" y="28.8099" size="0.02" layer="27" rot="R270"/>
 </element>
-<element name="R4" library="adafruit" package="M1206" value="10k" x="30.48" y="35.56" smashed="yes" rot="R180">
+<element name="R4" library="adafruit" package="M1206" value="UNUSED" x="30.48" y="35.56" smashed="yes" rot="R180">
 <attribute name="NAME" x="27.432" y="36.703" size="1.016" layer="25" font="vector" rot="R270"/>
-<attribute name="VALUE" x="26.797" y="36.068" size="1.27" layer="27" rot="R180"/>
+<attribute name="VALUE" x="33.782" y="37.973" size="1.27" layer="27" rot="R180"/>
 </element>
-<element name="R5" library="adafruit" package="M1206" value="10k" x="36.83" y="35.56" smashed="yes" rot="R180">
+<element name="R5" library="adafruit" package="M1206" value="UNUSED" x="36.83" y="35.56" smashed="yes" rot="R180">
 <attribute name="NAME" x="33.909" y="36.068" size="1.016" layer="25" font="vector" rot="R270"/>
-<attribute name="VALUE" x="33.02" y="35.941" size="1.27" layer="27" rot="R180"/>
+<attribute name="VALUE" x="40.64" y="37.846" size="1.27" layer="27" rot="R180"/>
 </element>
 <element name="Q1" library="transistor" package="TO92-EBC" value="BC349" x="41.91" y="26.797" smashed="yes" rot="R270">
@@
 <element name="R7" library="adafruit" package="M1206" value="10k" x="43.18" y="35.56" smashed="yes">
 <attribute name="NAME" x="41.656" y="34.798" size="1.016" layer="25" font="vector" rot="R90"/>
-<attribute name="VALUE" x="36.957" y="34.798" size="1.27" layer="27"/>
+<attribute name="VALUE" x="42.037" y="36.703" size="1.27" layer="27"/>
 </element>
 <element name="C1" library="adafruit" package="A/3216-18R" value="10uF" x="7.239" y="21.717" smashed="yes">
