File: eagle/modules/I2C/LCD-MCP23008/v1.1/lcd-i2c.sch (EAGLE design)
At the start: 18 parts, among them IC1 MCP2300X/P, J2 RJ12RIGHTANGLE-I2C, J3 RJ12RIGHTANGLE-I2C, Q1 BC349

Commit message: Update file and library
Parts:
- R4, R5: value 10k -> UNUSED
Changed lines of the file:
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@@
 <part name="A1" library="jumper" deviceset="SJ" device=""/>
 <part name="A0" library="jumper" deviceset="SJ" device=""/>
-<part name="R4" library="adafruit" deviceset="R-US_" device="M1206" value="10k"/>
-<part name="R5" library="adafruit" deviceset="R-US_" device="M1206" value="10k"/>
+<part name="R4" library="adafruit" deviceset="R-US_" device="M1206" value="UNUSED"/>
+<part name="R5" library="adafruit" deviceset="R-US_" device="M1206" value="UNUSED"/>
 <part name="P+6" library="supply1" deviceset="VCC" device=""/>
 <part name="P+7" library="supply1" deviceset="VCC" device=""/>
