File: eagle/modules/pico/v1.1/pico.brd (EAGLE design)
At the start: 93.3 x 53.3 mm, 45 parts, among them IC1 MEGA8-AI, IC3 ULN2803A, IC4 ULN2803A, J1 RS232, X1 16MHz

Commit message: Correct port numbering of pico
Parts:
- D2_IO3: value IO4 -> IO3
- D4_IO4: value IO3 -> IO4
- renumbered D2_IO4 to D2_IO3, D4_IO3 to D4_IO4
Changed lines of the file:
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@@
 <element name="IC3" library="lpatiny" package="SO18W" value="ULN2803A" x="72.39" y="26.035" rot="MR180"/>
 <element name="R3" library="resistor" package="M1206" value="1K" x="47.625" y="6.985" rot="MR90"/>
-<element name="D2_IO4" library="lpatiny" package="RJ12-STRAIGHT" value="IO4" x="55.88" y="38.1">
+<element name="D2_IO3" library="lpatiny" package="RJ12-STRAIGHT" value="IO3" x="55.88" y="38.1">
 <attribute name="OC_NEWARK" value="" x="-167.64" y="-41.91" size="1.778" layer="27" display="off"/>
 <attribute name="MPN" value="" x="-167.64" y="-41.91" size="1.778" layer="27" display="off"/>
@@
 </element>
 <element name="R0" library="resistor" package="M1206" value="1K" x="57.15" y="38.1" rot="MR270"/>
-<element name="D4_IO3" library="lpatiny" package="RJ12-STRAIGHT" value="IO3" x="72.39" y="38.1">
+<element name="D4_IO4" library="lpatiny" package="RJ12-STRAIGHT" value="IO4" x="72.39" y="38.1">
 <attribute name="OC_NEWARK" value="" x="-189.23" y="-59.69" size="1.778" layer="27" display="off"/>
 <attribute name="MPN" value="" x="-189.23" y="-59.69" size="1.778" layer="27" display="off"/>
@@
 <contactref element="J1" pad="GND1"/>
 <contactref element="J1" pad="GND2"/>
-<contactref element="D2_IO4" pad="GND1"/>
-<contactref element="D4_IO3" pad="GND1"/>
+<contactref element="D2_IO3" pad="GND1"/>
+<contactref element="D4_IO4" pad="GND1"/>
 <contactref element="IC4" pad="9"/>
 <contactref element="U$2" pad="GND2"/>
@@
 <contactref element="LED4" pad="K"/>
 <contactref element="I2C_INT0" pad="GND2"/>
-<contactref element="D2_IO4" pad="GND2"/>
-<contactref element="D4_IO3" pad="GND2"/>
+<contactref element="D2_IO3" pad="GND2"/>
+<contactref element="D4_IO4" pad="GND2"/>
 <contactref element="D9_IO2" pad="GND2"/>
 <contactref element="D10_IO1" pad="GND2"/>
@@
 <contactref element="I2C_INT0" pad="+12V"/>
 <contactref element="J1" pad="+12V"/>
-<contactref element="D2_IO4" pad="+12V"/>
-<contactref element="D4_IO3" pad="+12V"/>
+<contactref element="D2_IO3" pad="+12V"/>
+<contactref element="D4_IO4" pad="+12V"/>
 <wire x1="6.35" y1="1.27" x2="26.035" y2="1.27" width="1.778" layer="1"/>
 <wire x1="26.035" y1="1.27" x2="42.545" y2="1.27" width="1.778" layer="1"/>
@@
 </signal>
 <signal name="N$60" class="4">
-<contactref element="D2_IO4" pad="PWM"/>
+<contactref element="D2_IO3" pad="PWM"/>
 <contactref element="IC3" pad="14"/>
 <wire x1="54.6608" y1="44.5008" x2="54.0512" y2="44.5008" width="0.6096" layer="1"/>
@@
 </signal>
 <signal name="D2B6">
-<contactref element="D2_IO4" pad="I/O"/>
+<contactref element="D2_IO3" pad="I/O"/>
 <contactref element="R0" pad="1"/>
 <wire x1="57.0992" y1="42.0624" x2="57.0992" y2="39.624" width="0.4572" layer="16"/>
@@
 </signal>
 <signal name="D2B7">
-<contactref element="D4_IO3" pad="I/O"/>
+<contactref element="D4_IO4" pad="I/O"/>
 <contactref element="R1B" pad="1"/>
 <wire x1="73.5584" y1="39.624" x2="73.66" y2="39.5" width="0.4572" layer="16"/>
@@
 <signal name="N$2" class="4">
 <contactref element="IC3" pad="13"/>
-<contactref element="D4_IO3" pad="PWM"/>
+<contactref element="D4_IO4" pad="PWM"/>
 <wire x1="70.5104" y1="33.7312" x2="70.5104" y2="44.2976" width="0.6096" layer="16"/>
 <wire x1="70.5104" y1="26.0096" x2="70.5104" y2="33.7312" width="0.6096" layer="1"/>
@@
 <contactref element="I2C_INT0" pad="+5V"/>
 <contactref element="J1" pad="+5V"/>
-<contactref element="D2_IO4" pad="+5V"/>
-<contactref element="D4_IO3" pad="+5V"/>
+<contactref element="D2_IO3" pad="+5V"/>
+<contactref element="D4_IO4" pad="+5V"/>
 <wire x1="2.54" y1="50.8" x2="24.765" y2="50.8" width="1.778" layer="16"/>
 <wire x1="24.765" y1="50.8" x2="41.275" y2="50.8" width="1.778" layer="16"/>
