File: eagle/modules/femto/v1.1-unrouted-bad label/femto.brd (EAGLE design)
At the start: 50.2 x 25.1 mm, 29 parts, among them IC1 MEGA8-AI, J1 RJ12RIGHTANGLE-I2C, J2 RJ12RIGHTANGLE-I2C

Commit message: Correct femto
Parts:
- moved J1 3.81 mm to (45.7, 7.62), turned to 90 degrees
- moved C3 3.81 mm to (12.7, 14.6)
- moved J2 3.81 mm to (5.08, 7.62), turned to 270 degrees
- moved C1 3.81 mm to (12.7, 1.91)
- moved C2 3.81 mm to (12.7, 12.1)
Routing:
- net GND: track 118.1 -> 101.2 mm
- net 5V_B: track 89.0 -> 105.7 mm
- net N$13: track 58.4 -> 43.8 mm
- net SCK: track 0.00 -> 4.15 mm
- net N$4: track 0.76 -> 0.00 mm
