File: eagle/modules/I2C/LCD-atmega328/v1/lcd-i2c.sch (EAGLE design)
At the start: 19 parts, among them IC2 MEGA8-AI, J1 RJ12RIGHTANGLE-I2C, J4 RJ12RIGHTANGLE-I2C, Q1 BC349

Commit message: Correct LCD
Connections:
- removed net VCC: JP1.15, JP1.2, R6.A
- net +5V: now also JP1.15, JP1.2, R6.A
Changed lines of the file:
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@@
 </classes>
 <parts>
-<part name="P+4" library="supply1" deviceset="VCC" device=""/>
 <part name="GND4" library="supply1" deviceset="GND" device=""/>
-<part name="P+5" library="supply1" deviceset="VCC" device=""/>
 <part name="GND5" library="supply1" deviceset="GND" device=""/>
 <part name="R4" library="adafruit" deviceset="R-US_" device="M1206" value="EMPTY"/>
@@
 <part name="P+1" library="supply1" deviceset="+5V" device=""/>
 <part name="JP2" library="pinhead" deviceset="PINHD-2X10" device=""/>
+<part name="P+2" library="supply1" deviceset="+5V" device=""/>
+<part name="P+6" library="supply1" deviceset="+5V" device=""/>
 </parts>
 <sheets>
@@
 </plain>
 <instances>
-<instance part="P+4" gate="VCC" x="71.12" y="27.94"/>
 <instance part="GND4" gate="1" x="78.74" y="17.78"/>
-<instance part="P+5" gate="VCC" x="121.92" y="30.48" smashed="yes" rot="MR0">
-<attribute name="VALUE" x="127" y="30.48" size="1.778" layer="96" rot="MR0"/>
-</instance>
 <instance part="GND5" gate="1" x="96.52" y="27.94" rot="R180"/>
 <instance part="R4" gate="G$1" x="-58.42" y="-43.18" rot="MR90"/>
@@
 <instance part="P+1" gate="1" x="0" y="-35.56"/>
 <instance part="JP2" gate="A" x="111.76" y="71.12" rot="R180"/>
+<instance part="P+2" gate="1" x="68.58" y="27.94"/>
+<instance part="P+6" gate="1" x="121.92" y="30.48"/>
 </instances>
 <busses>
 </busses>
 <nets>
-<net name="VCC" class="1">
-<segment>
-<wire x1="71.12" y1="25.4" x2="73.66" y2="25.4" width="0.1524" layer="91"/>
-<wire x1="73.66" y1="38.1" x2="73.66" y2="25.4" width="0.1524" layer="91"/>
-<wire x1="73.66" y1="25.4" x2="88.9" y2="25.4" width="0.1524" layer="91"/>
-<wire x1="88.9" y1="25.4" x2="88.9" y2="20.32" width="0.1524" layer="91"/>
-<junction x="73.66" y="25.4"/>
-<pinref part="P+4" gate="VCC" pin="VCC"/>
-<pinref part="JP1" gate="A" pin="2"/>
-<pinref part="R6" gate="1" pin="A"/>
-</segment>
-<segment>
-<wire x1="121.92" y1="27.94" x2="121.92" y2="20.32" width="0.1524" layer="91"/>
-<pinref part="P+5" gate="VCC" pin="VCC"/>
-<pinref part="JP1" gate="A" pin="15"/>
-</segment>
-</net>
 <net name="GND" class="1">
 <segment>
@@
 <junction x="0" y="-38.1"/>
 </segment>
-</net>
+<segment>
+<wire x1="73.66" y1="38.1" x2="73.66" y2="25.4" width="0.1524" layer="91"/>
+<wire x1="73.66" y1="25.4" x2="88.9" y2="25.4" width="0.1524" layer="91"/>
+<wire x1="88.9" y1="25.4" x2="88.9" y2="20.32" width="0.1524" layer="91"/>
+<junction x="73.66" y="25.4"/>
+<pinref part="JP1" gate="A" pin="2"/>
+<pinref part="R6" gate="1" pin="A"/>
+<pinref part="P+2" gate="1" pin="+5V"/>
+<wire x1="73.66" y1="25.4" x2="68.58" y2="25.4" width="0.1524" layer="91"/>
+</segment>
+<segment>
+<pinref part="JP1" gate="A" pin="15"/>
+<pinref part="P+6" gate="1" pin="+5V"/>
+<wire x1="121.92" y1="20.32" x2="121.92" y2="27.94" width="0.1524" layer="91"/>
+</segment>
+</net>
