File: eagle/modules/pico/v2-atmega32u4-norouting/pico.sch (EAGLE design)
At the start: 54 parts, among them IC3 ULN2803A, IC4 ULN2803A, J1 RS232, U2 ATMEGA32U4-XUAU, X1 16MHz, X2 MINI-USB-UX60-MB-5ST

Commit message: Update
Parts:
- renumbered D10_IO1 to D4_IO1, D2_IO4 to D13_IO3, D4_IO3 to D6_IO4, D9_IO2 to D11_IO2, RGB1_D5-6-11 to RGB1_D6-9-10, RGB2_D7-8-13 to RGB2_D21-22-23
