File: eagle/modules/stepper/v1.0 - low curren - invertedt/stepper-v1.1.brd (EAGLE design)
At the start: 35.2 x 29.2 mm, 13 parts, among them IC1 ULN2803, IC3 CD74HC238M, J1 RJ12RIGHTANGLE

Commit message: Update stpeer low power
Parts:
- IC1: value ULN2803 -> (none)
- IC3: value CD74HC238M -> 74139; device lpatiny:SO16 -> lpatiny:SSOP08
- moved R5 12.0 mm to (8.89, 26.7), turned to 0 degrees
- moved IC3 3.81 mm to (8.89, 19.1)
Connections:
- net +5V: now also IC3.8; no longer IC3.16, IC3.6
- net GND: no longer IC3.3, IC3.5, IC3.8
- net N$1: now also IC3.7; no longer IC3.15
- net N$14: now also IC3.5; no longer IC3.13
- net N$7: now also IC3.3; no longer IC3.12
- net N$8: now also IC3.6; no longer IC3.14
Routing:
- net GND: track 33.3 -> 16.3 mm, vias 0 -> 1
- net N$2: track 32.3 -> 24.0 mm, vias 0 -> 2
- net N$13: track 23.6 -> 16.8 mm, vias 1 -> 0
- net +5V: track 65.1 -> 59.5 mm
- net N$1: track 8.98 -> 13.3 mm
- net N$8: track 8.37 -> 12.0 mm
- net N$14: track 8.98 -> 12.5 mm
- net N$7: track 9.41 -> 11.5 mm
- net N$4: track 34.1 -> 35.2 mm
