File: eagle/modules/femto/v2.0-unrouted/femto.sch (EAGLE design)
At the start: 29 parts, among them IC1 MEGA8-AI, J1 RJ12RIGHTANGLE-I2C, J2 RJ12RIGHTANGLE-I2C

Commit message: Update femto
Parts:
- added J3, J4, J5: RJ12RIGHTANGLE, lpatiny:RJ12RIGHTANGLE
Other:
- moved on the sheet: LED1, LED2, R1A, R1B, R1C, R2A, R2B, R2C
Changed lines of the file:
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@@
 <?xml version="1.0" encoding="utf-8"?>
 <!DOCTYPE eagle SYSTEM "eagle.dtd">
-<eagle version="6.4">
+<eagle version="6.1">
 <drawing>
 <settings>
@@
 <part name="R3" library="resistor" deviceset="R-EU_" device="M1206" value="1k"/>
 <part name="LED3" library="lpatiny" deviceset="LED3MM" device=""/>
+<part name="J3" library="lpatiny" deviceset="RJ12" device="RIGHTANGLE"/>
+<part name="J4" library="lpatiny" deviceset="RJ12" device="RIGHTANGLE"/>
+<part name="J5" library="lpatiny" deviceset="RJ12" device="RIGHTANGLE"/>
 </parts>
 <sheets>
@@
 <instance part="J2" gate="G$1" x="7.62" y="-33.02"/>
 <instance part="C3" gate="G$1" x="0" y="33.02" rot="R180"/>
-<instance part="LED2" gate="G$1" x="147.32" y="30.48" rot="R270"/>
-<instance part="LED1" gate="G$1" x="147.32" y="12.7" rot="R270"/>
-<instance part="R2A" gate="G$1" x="134.62" y="35.56"/>
-<instance part="R2B" gate="G$1" x="134.62" y="30.48"/>
-<instance part="R2C" gate="G$1" x="134.62" y="25.4"/>
-<instance part="R1A" gate="G$1" x="134.62" y="17.78"/>
-<instance part="R1B" gate="G$1" x="134.62" y="12.7"/>
-<instance part="R1C" gate="G$1" x="134.62" y="7.62"/>
-<instance part="GND7" gate="1" x="154.94" y="33.02"/>
-<instance part="GND8" gate="1" x="154.94" y="15.24"/>
+<instance part="LED2" gate="G$1" x="111.76" y="-5.08" rot="R270"/>
+<instance part="LED1" gate="G$1" x="111.76" y="-22.86" rot="R270"/>
+<instance part="R2A" gate="G$1" x="99.06" y="0"/>
+<instance part="R2B" gate="G$1" x="99.06" y="-5.08"/>
+<instance part="R2C" gate="G$1" x="99.06" y="-10.16"/>
+<instance part="R1A" gate="G$1" x="99.06" y="-17.78"/>
+<instance part="R1B" gate="G$1" x="99.06" y="-22.86"/>
+<instance part="R1C" gate="G$1" x="99.06" y="-27.94"/>
+<instance part="GND7" gate="1" x="119.38" y="-2.54"/>
+<instance part="GND8" gate="1" x="119.38" y="-20.32"/>
 <instance part="GND3" gate="1" x="114.3" y="12.7"/>
 <instance part="R6" gate="G$1" x="96.52" y="38.1"/>
@@
 <instance part="R3" gate="G$1" x="96.52" y="35.56"/>
 <instance part="LED3" gate="G$1" x="109.22" y="35.56" rot="R90"/>
+<instance part="J3" gate="G$1" x="132.08" y="86.36"/>
+<instance part="J4" gate="G$1" x="132.08" y="68.58"/>
+<instance part="J5" gate="G$1" x="132.08" y="48.26"/>
 </instances>
 <busses>
@@
 <segment>
 <pinref part="LED2" gate="G$1" pin="A2"/>
-<wire x1="149.86" y1="35.56" x2="154.94" y2="35.56" width="0.1524" layer="91"/>
+<wire x1="114.3" y1="0" x2="119.38" y2="0" width="0.1524" layer="91"/>
 <pinref part="GND7" gate="1" pin="GND"/>
 </segment>
 <segment>
 <pinref part="LED1" gate="G$1" pin="A2"/>
-<wire x1="149.86" y1="17.78" x2="154.94" y2="17.78" width="0.1524" layer="91"/>
+<wire x1="114.3" y1="-17.78" x2="119.38" y2="-17.78" width="0.1524" layer="91"/>
 <pinref part="GND8" gate="1" pin="GND"/>
 </segment>
@@
 <segment>
 <pinref part="R1B" gate="G$1" pin="1"/>
-<wire x1="129.54" y1="12.7" x2="127" y2="12.7" width="0.1524" layer="91"/>
-<label x="125.73" y="13.462" size="1.27" layer="95"/>
+<wire x1="93.98" y1="-22.86" x2="91.44" y2="-22.86" width="0.1524" layer="91"/>
+<label x="90.17" y="-22.098" size="1.27" layer="95"/>
 </segment>
 <segment>
@@
 <segment>
 <pinref part="R2B" gate="G$1" pin="1"/>
-<wire x1="129.54" y1="30.48" x2="127" y2="30.48" width="0.1524" layer="91"/>
-<label x="125.73" y="30.988" size="1.27" layer="95"/>
+<wire x1="93.98" y1="-5.08" x2="91.44" y2="-5.08" width="0.1524" layer="91"/>
+<label x="90.17" y="-4.572" size="1.27" layer="95"/>
 </segment>
 <segment>
@@
 <pinref part="R2A" gate="G$1" pin="2"/>
 <pinref part="LED2" gate="G$1" pin="CRED"/>
-<wire x1="142.24" y1="35.56" x2="139.7" y2="35.56" width="0.1524" layer="91"/>
+<wire x1="106.68" y1="0" x2="104.14" y2="0" width="0.1524" layer="91"/>
 </segment>
 </net>
@@
 <pinref part="LED2" gate="G$1" pin="CBLUE"/>
 <pinref part="R2B" gate="G$1" pin="2"/>
-<wire x1="142.24" y1="30.48" x2="139.7" y2="30.48" width="0.1524" layer="91"/>
+<wire x1="106.68" y1="-5.08" x2="104.14" y2="-5.08" width="0.1524" layer="91"/>
 </segment>
 </net>
@@
 <pinref part="R2C" gate="G$1" pin="2"/>
 <pinref part="LED2" gate="G$1" pin="CGREEN"/>
-<wire x1="142.24" y1="25.4" x2="139.7" y2="25.4" width="0.1524" layer="91"/>
+<wire x1="106.68" y1="-10.16" x2="104.14" y2="-10.16" width="0.1524" layer="91"/>
 </segment>
 </net>
@@
 <pinref part="LED1" gate="G$1" pin="CRED"/>
 <pinref part="R1A" gate="G$1" pin="2"/>
-<wire x1="142.24" y1="17.78" x2="139.7" y2="17.78" width="0.1524" layer="91"/>
+<wire x1="106.68" y1="-17.78" x2="104.14" y2="-17.78" width="0.1524" layer="91"/>
 </segment>
 </net>
@@
 <pinref part="R1B" gate="G$1" pin="2"/>
 <pinref part="LED1" gate="G$1" pin="CBLUE"/>
-<wire x1="142.24" y1="12.7" x2="139.7" y2="12.7" width="0.1524" layer="91"/>
+<wire x1="106.68" y1="-22.86" x2="104.14" y2="-22.86" width="0.1524" layer="91"/>
 </segment>
 </net>
@@
 <pinref part="LED1" gate="G$1" pin="CGREEN"/>
 <pinref part="R1C" gate="G$1" pin="2"/>
-<wire x1="142.24" y1="7.62" x2="139.7" y2="7.62" width="0.1524" layer="91"/>
+<wire x1="106.68" y1="-27.94" x2="104.14" y2="-27.94" width="0.1524" layer="91"/>
 </segment>
 </net>
@@
 <segment>
 <pinref part="R2A" gate="G$1" pin="1"/>
-<wire x1="129.54" y1="35.56" x2="127" y2="35.56" width="0.1524" layer="91"/>
-<label x="125.476" y="36.322" size="1.27" layer="95"/>
+<wire x1="93.98" y1="0" x2="91.44" y2="0" width="0.1524" layer="91"/>
+<label x="89.916" y="0.762" size="1.27" layer="95"/>
 </segment>
 <segment>
@@
 <segment>
 <pinref part="R2C" gate="G$1" pin="1"/>
-<wire x1="129.54" y1="25.4" x2="127" y2="25.4" width="0.1524" layer="91"/>
-<label x="125.476" y="26.416" size="1.27" layer="95"/>
+<wire x1="93.98" y1="-10.16" x2="91.44" y2="-10.16" width="0.1524" layer="91"/>
+<label x="89.916" y="-9.144" size="1.27" layer="95"/>
 </segment>
 </net>
@@
 <segment>
 <pinref part="R1A" gate="G$1" pin="1"/>
-<wire x1="129.54" y1="17.78" x2="127" y2="17.78" width="0.1524" layer="91"/>
-<label x="125.984" y="18.796" size="1.27" layer="95"/>
+<wire x1="93.98" y1="-17.78" x2="91.44" y2="-17.78" width="0.1524" layer="91"/>
+<label x="90.424" y="-16.764" size="1.27" layer="95"/>
 </segment>
 <segment>
@@
 <segment>
 <pinref part="R1C" gate="G$1" pin="1"/>
-<wire x1="129.54" y1="7.62" x2="127" y2="7.62" width="0.1524" layer="91"/>
-<label x="126.238" y="8.128" size="1.27" layer="95"/>
-</segment>
-</net>
+<wire x1="93.98" y1="-27.94" x2="91.44" y2="-27.94" width="0.1524" layer="91"/>
+<label x="90.678" y="-27.432" size="1.27" layer="95"/>
+</segment>
+</net>

Commit message: Update stepper demo for LOW intensity module
Parts:
- added IC2: (no value), lpatiny:ULN2803A
Connections:
- removed net N$13: J1.1, J2.1
- new net +12V: J1.1, J2.1, J3.1, J4.1, J5.1
- new net N$3: IC2.O1, IC2.O2, IC2.O3, J3.2
- new net N$5: IC2.O4, IC2.O5, J4.2
- new net N$6: IC2.O6, IC2.O7, IC2.O8, J5.2
- net 5V_B: now also J3.5, J4.5, J5.5
- net A0: now also IC2.I1, IC2.I2, IC2.I3
- net A1: now also J3.3
- net A2: now also IC2.I4, IC2.I5
- net A3: now also J4.3
- net A6: now also IC2.I6, IC2.I7, IC2.I8
- net A7: now also J5.3
- net GND: now also IC2.GND, J3.4, J3.6, J4.4, J4.6, J5.4, J5.6
Other:
- moved on the sheet: J3, J4, J5
Changed lines of the file:
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@@
 <?xml version="1.0" encoding="utf-8"?>
 <!DOCTYPE eagle SYSTEM "eagle.dtd">
-<eagle version="6.1">
+<eagle version="6.4">
 <drawing>
 <settings>
@@
 <part name="J4" library="lpatiny" deviceset="RJ12" device="RIGHTANGLE"/>
 <part name="J5" library="lpatiny" deviceset="RJ12" device="RIGHTANGLE"/>
+<part name="IC2" library="lpatiny" deviceset="ULN2803A" device=""/>
+<part name="GND4" library="supply1" deviceset="GND" device=""/>
+<part name="GND11" library="supply1" deviceset="GND" device=""/>
+<part name="GND12" library="supply1" deviceset="GND" device=""/>
+<part name="GND13" library="supply1" deviceset="GND" device=""/>
 </parts>
 <sheets>
@@
 <instance part="R3" gate="G$1" x="96.52" y="35.56"/>
 <instance part="LED3" gate="G$1" x="109.22" y="35.56" rot="R90"/>
-<instance part="J3" gate="G$1" x="132.08" y="86.36"/>
-<instance part="J4" gate="G$1" x="132.08" y="68.58"/>
-<instance part="J5" gate="G$1" x="132.08" y="48.26"/>
+<instance part="J3" gate="G$1" x="162.56" y="99.06"/>
+<instance part="J4" gate="G$1" x="162.56" y="76.2"/>
+<instance part="J5" gate="G$1" x="162.56" y="53.34"/>
+<instance part="IC2" gate="G$1" x="114.3" y="71.12"/>
+<instance part="GND4" gate="1" x="101.6" y="50.8"/>
+<instance part="GND11" gate="1" x="144.78" y="43.18"/>
+<instance part="GND12" gate="1" x="144.78" y="66.04"/>
+<instance part="GND13" gate="1" x="144.78" y="88.9"/>
 </instances>
 <busses>
@@
 <pinref part="GND10" gate="1" pin="GND"/>
 </segment>
+<segment>
+<pinref part="IC2" gate="G$1" pin="GND"/>
+<pinref part="GND4" gate="1" pin="GND"/>
+<wire x1="101.6" y1="60.96" x2="101.6" y2="53.34" width="0.1524" layer="91"/>
+</segment>
+<segment>
+<pinref part="J5" gate="G$1" pin="6"/>
+<pinref part="J5" gate="G$1" pin="4"/>
+<wire x1="160.02" y1="50.8" x2="144.78" y2="50.8" width="0.1524" layer="91"/>
+<wire x1="144.78" y1="50.8" x2="144.78" y2="45.72" width="0.1524" layer="91"/>
+<wire x1="144.78" y1="45.72" x2="160.02" y2="45.72" width="0.1524" layer="91"/>
+<pinref part="GND11" gate="1" pin="GND"/>
+<junction x="144.78" y="45.72"/>
+</segment>
+<segment>
+<pinref part="J4" gate="G$1" pin="4"/>
+<wire x1="160.02" y1="73.66" x2="144.78" y2="73.66" width="0.1524" layer="91"/>
+<wire x1="144.78" y1="73.66" x2="144.78" y2="68.58" width="0.1524" layer="91"/>
+<pinref part="J4" gate="G$1" pin="6"/>
+<wire x1="144.78" y1="68.58" x2="160.02" y2="68.58" width="0.1524" layer="91"/>
+<pinref part="GND12" gate="1" pin="GND"/>
+<junction x="144.78" y="68.58"/>
+</segment>
+<segment>
+<pinref part="J3" gate="G$1" pin="4"/>
+<wire x1="160.02" y1="96.52" x2="144.78" y2="96.52" width="0.1524" layer="91"/>
+<wire x1="144.78" y1="96.52" x2="144.78" y2="91.44" width="0.1524" layer="91"/>
+<pinref part="J3" gate="G$1" pin="6"/>
+<wire x1="144.78" y1="91.44" x2="160.02" y2="91.44" width="0.1524" layer="91"/>
+<pinref part="GND13" gate="1" pin="GND"/>
+<junction x="144.78" y="91.44"/>
+</segment>
 </net>
 <net name="A0" class="0">
 <segment>
 <pinref part="IC1" gate="G$1" pin="PC0(ADC0)"/>
-<wire x1="83.82" y1="68.58" x2="91.44" y2="68.58" width="0.1524" layer="91"/>
+<wire x1="83.82" y1="68.58" x2="93.98" y2="68.58" width="0.1524" layer="91"/>
 <label x="90.424" y="69.088" size="1.016" layer="95"/>
+<wire x1="93.98" y1="68.58" x2="93.98" y2="76.2" width="0.1524" layer="91"/>
+<pinref part="IC2" gate="G$1" pin="I3"/>
+<wire x1="93.98" y1="76.2" x2="101.6" y2="76.2" width="0.1524" layer="91"/>
+<pinref part="IC2" gate="G$1" pin="I2"/>
+<wire x1="101.6" y1="76.2" x2="101.6" y2="78.74" width="0.1524" layer="91"/>
+<pinref part="IC2" gate="G$1" pin="I1"/>
+<wire x1="101.6" y1="78.74" x2="101.6" y2="81.28" width="0.1524" layer="91"/>
+<junction x="101.6" y="81.28"/>
+<junction x="101.6" y="78.74"/>
+<junction x="101.6" y="76.2"/>
 </segment>
 </net>
@@
 <label x="90.17" y="61.722" size="1.016" layer="95"/>
 </segment>
+<segment>
+<pinref part="J4" gate="G$1" pin="3"/>
+<wire x1="160.02" y1="76.2" x2="152.4" y2="76.2" width="0.1524" layer="91"/>
+<label x="151.892" y="76.454" size="1.016" layer="95"/>
+</segment>
 </net>
 <net name="A2" class="0">
 <segment>
 <pinref part="IC1" gate="G$1" pin="PC2(ADC2)"/>
-<wire x1="91.44" y1="63.5" x2="83.82" y2="63.5" width="0.1524" layer="91"/>
 <label x="90.17" y="64.008" size="1.016" layer="95"/>
+<wire x1="83.82" y1="63.5" x2="96.52" y2="63.5" width="0.1524" layer="91"/>
+<wire x1="96.52" y1="63.5" x2="96.52" y2="71.12" width="0.1524" layer="91"/>
+<pinref part="IC2" gate="G$1" pin="I5"/>
+<wire x1="96.52" y1="71.12" x2="101.6" y2="71.12" width="0.1524" layer="91"/>
+<pinref part="IC2" gate="G$1" pin="I4"/>
+<wire x1="101.6" y1="71.12" x2="101.6" y2="73.66" width="0.1524" layer="91"/>
+<junction x="101.6" y="73.66"/>
+<junction x="101.6" y="71.12"/>
 </segment>
 </net>
@@
 <label x="90.424" y="66.548" size="1.016" layer="95"/>
 </segment>
+<segment>
+<pinref part="J3" gate="G$1" pin="3"/>
+<wire x1="160.02" y1="99.06" x2="152.4" y2="99.06" width="0.1524" layer="91"/>
+<label x="151.892" y="99.314" size="1.016" layer="95"/>
+</segment>
 </net>
 <net name="SCK" class="0">
@@
 </segment>
 </net>
-<net name="N$13" class="0">
+<net name="+12V" class="0">
 <segment>
 <pinref part="J1" gate="G$1" pin="1"/>
@@
 <junction x="5.08" y="-27.94"/>
 <label x="-9.398" y="-26.924" size="1.778" layer="95"/>
+</segment>
+<segment>
+<pinref part="J3" gate="G$1" pin="1"/>
+<wire x1="160.02" y1="104.14" x2="152.4" y2="104.14" width="0.1524" layer="91"/>
+<label x="151.638" y="104.394" size="1.016" layer="95"/>
+</segment>
+<segment>
+<pinref part="J4" gate="G$1" pin="1"/>
+<wire x1="160.02" y1="81.28" x2="152.4" y2="81.28" width="0.1524" layer="91"/>
+<label x="151.638" y="81.534" size="1.016" layer="95"/>
+</segment>
+<segment>
+<pinref part="J5" gate="G$1" pin="1"/>
+<wire x1="160.02" y1="58.42" x2="152.4" y2="58.42" width="0.1524" layer="91"/>
+<label x="151.892" y="58.928" size="1.016" layer="95"/>
 </segment>
 </net>
@@
 <label x="-13.462" y="21.082" size="1.778" layer="95"/>
 </segment>
+<segment>
+<pinref part="J3" gate="G$1" pin="5"/>
+<wire x1="160.02" y1="93.98" x2="152.4" y2="93.98" width="0.1524" layer="91"/>
+<label x="151.892" y="94.234" size="1.016" layer="95"/>
+</segment>
+<segment>
+<pinref part="J4" gate="G$1" pin="5"/>
+<wire x1="160.02" y1="71.12" x2="152.4" y2="71.12" width="0.1524" layer="91"/>
+<label x="151.638" y="71.374" size="1.016" layer="95"/>
+</segment>
+<segment>
+<pinref part="J5" gate="G$1" pin="5"/>
+<wire x1="160.02" y1="48.26" x2="152.4" y2="48.26" width="0.1524" layer="91"/>
+<label x="151.638" y="48.768" size="1.016" layer="95"/>
+</segment>
 </net>
 <net name="N$16" class="0">
@@
 <segment>
 <pinref part="IC1" gate="G$1" pin="ADC6"/>
-<wire x1="83.82" y1="53.34" x2="91.44" y2="53.34" width="0.1524" layer="91"/>
 <label x="90.424" y="53.848" size="1.016" layer="95"/>
+<wire x1="83.82" y1="53.34" x2="99.06" y2="53.34" width="0.1524" layer="91"/>
+<wire x1="99.06" y1="53.34" x2="99.06" y2="63.5" width="0.1524" layer="91"/>
+<pinref part="IC2" gate="G$1" pin="I8"/>
+<wire x1="99.06" y1="63.5" x2="101.6" y2="63.5" width="0.1524" layer="91"/>
+<pinref part="IC2" gate="G$1" pin="I7"/>
+<wire x1="101.6" y1="63.5" x2="101.6" y2="66.04" width="0.1524" layer="91"/>
+<pinref part="IC2" gate="G$1" pin="I6"/>
+<wire x1="101.6" y1="66.04" x2="101.6" y2="68.58" width="0.1524" layer="91"/>
+<junction x="101.6" y="68.58"/>
+<junction x="101.6" y="66.04"/>
+<junction x="101.6" y="63.5"/>
 </segment>
 </net>
@@
 <label x="90.424" y="51.054" size="1.016" layer="95"/>
 </segment>
-</net>
+<segment>
+<pinref part="J5" gate="G$1" pin="3"/>
+<wire x1="160.02" y1="53.34" x2="152.4" y2="53.34" width="0.1524" layer="91"/>
+<label x="152.146" y="53.848" size="1.016" layer="95"/>
+</segment>
+</net>
+<net name="N$3" class="0">
+<segment>
+<pinref part="IC2" gate="G$1" pin="O1"/>
+<pinref part="IC2" gate="G$1" pin="O2"/>
+<wire x1="127" y1="81.28" x2="127" y2="78.74" width="0.1524" layer="91"/>
+<pinref part="IC2" gate="G$1" pin="O3"/>
+<wire x1="127" y1="78.74" x2="127" y2="76.2" width="0.1524" layer="91"/>
+<wire x1="127" y1="76.2" x2="134.62" y2="76.2" width="0.1524" layer="91"/>
+<wire x1="134.62" y1="76.2" x2="134.62" y2="101.6" width="0.1524" layer="91"/>
+<pinref part="J3" gate="G$1" pin="2"/>
+<wire x1="134.62" y1="101.6" x2="160.02" y2="101.6" width="0.1524" layer="91"/>
+<junction x="127" y="76.2"/>
+<junction x="127" y="78.74"/>
+<junction x="127" y="81.28"/>
+</segment>
+</net>
+<net name="N$5" class="0">
+<segment>
+<pinref part="J4" gate="G$1" pin="2"/>
+<wire x1="160.02" y1="78.74" x2="137.16" y2="78.74" width="0.1524" layer="91"/>
+<wire x1="137.16" y1="78.74" x2="137.16" y2="73.66" width="0.1524" layer="91"/>
+<pinref part="IC2" gate="G$1" pin="O4"/>
+<wire x1="137.16" y1="73.66" x2="127" y2="73.66" width="0.1524" layer="91"/>
+<pinref part="IC2" gate="G$1" pin="O5"/>
+<wire x1="127" y1="73.66" x2="127" y2="71.12" width="0.1524" layer="91"/>
+<junction x="127" y="71.12"/>
+<junction x="127" y="73.66"/>
+</segment>
+</net>
+<net name="N$6" class="0">
+<segment>
+<pinref part="J5" gate="G$1" pin="2"/>
+<wire x1="160.02" y1="55.88" x2="134.62" y2="55.88" width="0.1524" layer="91"/>
+<wire x1="134.62" y1="55.88" x2="134.62" y2="63.5" width="0.1524" layer="91"/>
+<pinref part="IC2" gate="G$1" pin="O8"/>
+<wire x1="134.62" y1="63.5" x2="127" y2="63.5" width="0.1524" layer="91"/>
+<pinref part="IC2" gate="G$1" pin="O7"/>
+<wire x1="127" y1="63.5" x2="127" y2="66.04" width="0.1524" layer="91"/>
+<pinref part="IC2" gate="G$1" pin="O6"/>
+<wire x1="127" y1="66.04" x2="127" y2="68.58" width="0.1524" layer="91"/>
+<junction x="127" y="68.58"/>
+<junction x="127" y="66.04"/>
+<junction x="127" y="63.5"/>
+</segment>
+</net>
