File: eagle/halloween2013/10-io/femto.brd (EAGLE design)
At the start: 48.9 x 49.2 mm, 16 parts, among them IC1 MEGA8-AI, J1 RJ12RIGHTANGLE-I2C, J2 RJ12RIGHTANGLE-I2C

Commit message: Update halloween
Parts:
- removed X6, X7, X8, X9: (no value), con-molex:22-23-2061
- added C5, C7: 10uF, rcl:C1206
- added IC2, IC3: (no value), lpatiny:SO18W
- added J10, J11, J12, J3, J4, J5, J6, J7, J8, J9: RJ12RIGHTANGLE, lpatiny:RJ12-RIGHTANGLE
- added JP1: (no value), SparkFun:SCREWTERMINAL-3.5MM-2
- added R2A1, R2A10, R2A2, R2A3, R2A4, R2A5, R2A6, R2A7, R2A8, R2A9: 1k, resistor:M1206
- added U$1: KPJX-4S-S, lpatiny:KPJX-4S-S
- added X1: 87758-0616, con-molex:87758-0616
- moved J2 74.9 mm to (83.8, 24.1)
- moved CON2 49.1 mm to (83.8, 57.8), flipped to the bottom, turned to 270 degrees
- moved J1 46.2 mm to (83.8, 39.4), turned to 90 degrees
- moved C1 26.9 mm to (52.1, 41.3), flipped to the bottom
- moved C2 26.9 mm to (45.7, 41.3), flipped to the bottom, turned to 180 degrees
- moved LED7 24.0 mm to (51.4, 26.0)
- moved R7 24.0 mm to (48.3, 26.0)
- moved C3 19.7 mm to (39.4, 41.3), flipped to the bottom, turned to 180 degrees
- moved D1 18.8 mm to (29.5, 43.2), flipped to the bottom, turned to 270 degrees
- moved D2 17.2 mm to (29.5, 43.2), turned to 270 degrees
- moved IC1 16.6 mm to (39.4, 31.8), flipped to the bottom, turned to 0 degrees
- moved R8 7.01 mm to (26.0, 43.2), flipped to the bottom, turned to 90 degrees
Connections:
- removed net D0: IC1.30, X6.1
- removed net D1: IC1.31, X6.2
- removed net PB6: IC1.7, X8.5
- removed net PB7: IC1.8, X9.5
- new net +12V: J10.+12V, J11.+12V, J12.+12V, J3.+12V, J4.+12V, J5.+12V, J6.+12V, J7.+12V, J8.+12V, J9.+12V
- new net EXT-12V: C7.2, U$1.+12V, X1.2
- new net EXT-5V: C5.1, U$1.+5V, X1.1
- new net I2C-12V: J1.+12V, J2.+12V, X1.6
- new net I2C-5V: D2.A, J1.+5V, J2.+5V, X1.5
- new net N$1: IC2.1, IC2.2
- new net N$10: J5.I/O, R2A3.2
- new net N$11: IC2.12, J6.PWM
- new net N$12: J6.I/O, R2A4.2
- new net N$14: J7.I/O, R2A5.2
- new net N$16: IC2.7
- new net N$17: IC2.8
- new net N$18: IC3.17, IC3.18, J8.PWM
- new net N$19: IC3.15, IC3.16, J9.PWM
- new net N$2: J3.I/O, R2A1.2
- new net N$20: IC3.13, IC3.14, J10.PWM
- new net N$21: J8.I/O, R2A6.2
- new net N$22: J9.I/O, R2A7.2
- new net N$23: J10.I/O, R2A8.2
- new net N$24: IC3.12, J11.PWM
- new net N$25: J11.I/O, R2A9.2
- new net N$26: IC3.11, J12.PWM
- new net N$27: J12.I/O, R2A10.2
- new net N$28: IC3.1, IC3.2
- new net N$29: IC3.3, IC3.4
- new net N$3: IC2.17, IC2.18, J3.PWM
- new net N$30: IC3.5, IC3.6
- new net N$31: IC3.7
- new net N$32: IC3.8
- new net N$37: X1.4
- new net N$38: X1.3
- new net N$5: IC2.15, IC2.16, J4.PWM
- new net N$6: IC2.13, IC2.14, J5.PWM
- new net N$7: IC2.3, IC2.4
- new net N$8: IC2.5, IC2.6
- new net N$9: J4.I/O, R2A2.2
- new net RX: IC1.30
- new net TX: IC1.31
- net 5V_B: now also J10.+5V, J11.+5V, J12.+5V, J3.+5V, J4.+5V, J5.+5V, J6.+5V, J7.+5V, J8.+5V, J9.+5V, JP1.1; no longer D2.A, J1.+5V, J2.+5V
- net A0: no longer X9.1
- net A1: no longer X9.2
- net A2: no longer X9.3
- net A3: now also R2A1.1, R2A6.1; no longer X9.4
- net D10: no longer X8.1
- net D2: now also R2A2.1, R2A7.1; no longer X6.3
- net D3: no longer X6.4
- net D4: no longer X6.5
- net D5: no longer X7.1
- net D6: no longer X7.2
- net D7: no longer X7.3
- net D8: no longer X7.4
- net D9: no longer X7.5
- net GND: now also C5.2, C7.1, IC2.9, IC3.9, J10.GND1, J10.GND2, J11.GND1, J11.GND2, J12.GND1, J12.GND2, J3.GND1, J3.GND2, J4.GND1, J4.GND2, J5.GND1, J5.GND2, J6.GND1, J6.GND2, J7.GND1, J7.GND2, J8.GND1, J8.GND2, J9.GND1, J9.GND2, JP1.2, U$1.GND1, U$1.GND2; no longer X6.6, X7.6, X8.6, X9.6
- net MISO: now also R2A10.1, R2A3.1, R2A4.1, R2A5.1, R2A8.1, R2A9.1; no longer X8.3
- net MOSI: no longer X8.2
- net N$13: now also IC2.11, J7.PWM; no longer J1.+12V, J2.+12V
- net SCK: no longer X8.4
Routing:
- net MOSI: track 3.89 -> 0.00 mm
- net SCK: track 3.57 -> 0.00 mm
- net 5V_A: track 2.99 -> 0.00 mm
- net MISO: track 2.99 -> 0.00 mm
- net GND: track 2.11 -> 0.00 mm
- net RESET: track 1.66 -> 0.00 mm
Other:
- board size 48.9 x 49.2 mm -> 88.9 x 63.2 mm
- board text removed: "D0"
