File: eagle/halloween/halloween2013/10-io/v-norouting/femto.sch (EAGLE design)
At the start: 39 parts, among them IC1 MEGA8-AI, J1 RJ12RIGHTANGLE-I2C, J10 RJ12RIGHTANGLE, J11 RJ12RIGHTANGLE, J12 RJ12RIGHTANGLE, J2 RJ12RIGHTANGLE-I2C, J3 RJ12RIGHTANGLE, J4 RJ12RIGHTANGLE, J5 RJ12RIGHTANGLE, J6 RJ12RIGHTANGLE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

Commit message: Update halloween
Connections:
- net 5V_A renamed 5V_ISCP
- removed net 5V_B: J10.5, J11.5, J12.5, J3.5, J4.5, J5.5, J6.5, J7.5, J8.5, J9.5, X1-3.S
- removed net N$1: IC2.I1, IC2.I2
- removed net N$16: IC2.I7
- removed net N$17: IC2.I8
- removed net N$28: IC3.I1, IC3.I2
- removed net N$29: IC3.I3, IC3.I4
- removed net N$30: IC3.I5, IC3.I6
- removed net N$31: IC3.I7
- removed net N$32: IC3.I8
- removed net N$7: IC2.I3, IC2.I4
- removed net N$8: IC2.I5, IC2.I6
- removed net RX: IC1.PD0(RXD)
- removed net TX: IC1.PD1(TXD)
- new net 5V_UC: C1.1, C2.1, C3.1, D1.C, D2.C, D3.C, IC1.AVCC, IC1.VCC@1, IC1.VCC@2, R7.1, R8.2
- new net D0: IC1.PD0(RXD), IC2.I1, IC2.I2
- new net D1: IC1.PD1(TXD), IC2.I3, IC2.I4
- new net PB6: IC1.PB6(XTAL1/TOSC1), R2A5.1
- new net PB7: IC1.PB7(XTAL2/TOSC2), R2A10.1
- net +12V: now also C7.1
- net +5V: now also C5.1, J10.5, J11.5, J12.5, J3.5, J4.5, J5.5, J6.5, J7.5, J8.5, J9.5, X1-3.S; no longer C1.1, C2.1, C3.1, D1.C, D2.C, D3.C, IC1.AVCC, IC1.VCC@1, IC1.VCC@2, R7.1, R8.2
- net A0: now also R2A6.1
- net A1: now also R2A7.1
- net A2: now also R2A8.1
- net A3: now also R2A9.1; no longer R2A1.1, R2A6.1
- net D10: now also R2A1.1
- net D2: now also IC2.I5, IC2.I6; no longer R2A2.1, R2A7.1
- net D3: now also IC2.I7
- net D4: now also IC2.I8
- net D5: now also IC3.I1, IC3.I2
- net D6: now also IC3.I3, IC3.I4
- net D7: now also IC3.I5, IC3.I6
- net D8: now also IC3.I7
- net D9: now also IC3.I8
- net EXT-12V: no longer C7.2
- net EXT-5V: no longer C5.1
- net GND: now also C7.2; no longer C7.1
- net MISO: no longer R2A10.1, R2A4.1, R2A5.1, R2A8.1, R2A9.1
- net MOSI: now also R2A2.1
- net SCK: now also R2A4.1
Other:
- moved on the sheet: C5, C7
