File: eagle/halloween/halloween2013/10-io/v1/femto.brd (EAGLE design)
At the start: 88.9 x 63.2 mm, 39 parts, among them IC1 MEGA8-AI, J1 RJ12RIGHTANGLE-I2C, J10 RJ12RIGHTANGLE, J11 RJ12RIGHTANGLE, J12 RJ12RIGHTANGLE, J2 RJ12RIGHTANGLE-I2C, J3 RJ12RIGHTANGLE, J4 RJ12RIGHTANGLE, J5 RJ12RIGHTANGLE, J6 RJ12RIGHTANGLE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

Commit message: Update halloween
Parts:
- moved CON2 62.5 mm to (27.9, 29.8), turned to 90 degrees
- moved C7 21.6 mm to (7.62, 20.3), flipped to the bottom, turned to 0 degrees
- moved C1 20.1 mm to (35.6, 29.8)
- moved C5 18.9 mm to (7.62, 43.2), flipped to the bottom
- moved LED7 15.5 mm to (36.2, 23.5)
- moved R7 15.5 mm to (33.0, 23.5)
- moved D3 14.5 mm to (35.6, 36.8)
- moved D1 14.3 mm to (35.6, 30.2), flipped to the top, turned to 0 degrees
- moved C2 13.5 mm to (35.6, 32.4)
- moved D2 11.5 mm to (35.6, 33.3), turned to 0 degrees
- moved R8 11.1 mm to (35.6, 37.5), turned to 0 degrees
- moved X1 10.2 mm to (17.8, 31.8), flipped to the bottom, turned to 180 degrees
- moved IC1 7.62 mm to (47.0, 31.8)
- moved C3 7.41 mm to (35.6, 34.9)
- moved R2A1 2.84 mm to (11.4, 45.7), turned to 180 degrees
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Connections:
- net 5V_A renamed 5V_ISCP
- removed net 5V_B: J10.+5V, J11.+5V, J12.+5V, J3.+5V, J4.+5V, J5.+5V, J6.+5V, J7.+5V, J8.+5V, J9.+5V, X1.3
- removed net N$1: IC2.1, IC2.2
- removed net N$16: IC2.7
- removed net N$17: IC2.8
- removed net N$28: IC3.1, IC3.2
- removed net N$29: IC3.3, IC3.4
- removed net N$30: IC3.5, IC3.6
- removed net N$31: IC3.7
- removed net N$32: IC3.8
- removed net N$7: IC2.3, IC2.4
- removed net N$8: IC2.5, IC2.6
- removed net RX: IC1.30
- removed net TX: IC1.31
- new net 5V_UC: C1.1, C2.1, C3.1, D1.C, D2.C, D3.C, IC1.18, IC1.4, IC1.6, R7.1, R8.2
- new net D0: IC1.30, IC2.1, IC2.2
- new net D1: IC1.31, IC2.3, IC2.4
- new net PB6: IC1.7, R2A5.1
- new net PB7: IC1.8, R2A10.1
- net +12V: now also C7.1
- net +5V: now also C5.1, J10.+5V, J11.+5V, J12.+5V, J3.+5V, J4.+5V, J5.+5V, J6.+5V, J7.+5V, J8.+5V, J9.+5V, X1.3; no longer C1.1, C2.1, C3.1, D1.C, D2.C, D3.C, IC1.18, IC1.4, IC1.6, R7.1, R8.2
- net A0: now also R2A6.1
- net A1: now also R2A7.1
- net A2: now also R2A8.1
- net A3: now also R2A9.1; no longer R2A1.1, R2A6.1
- net D10: now also R2A1.1
- net D2: now also IC2.5, IC2.6; no longer R2A2.1, R2A7.1
- net D3: now also IC2.7
- net D4: now also IC2.8
- net D5: now also IC3.1, IC3.2
- net D6: now also IC3.3, IC3.4
- net D7: now also IC3.5, IC3.6
- net D8: now also IC3.7
- net D9: now also IC3.8
- net EXT-12V: no longer C7.2
- net EXT-5V: no longer C5.1
- net GND: now also C7.2; no longer C7.1
- net MISO: no longer R2A10.1, R2A4.1, R2A5.1, R2A8.1, R2A9.1
- net MOSI: now also R2A2.1
- net SCK: now also R2A4.1
Routing:
- net +5V: track 0.00 -> 257.8 mm
- net I2C-5V: track 0.00 -> 113.1 mm, vias 0 -> 1
- net GND: track 417.5 -> 512.3 mm, vias 0 -> 3
- net N$19: track 0.00 -> 73.8 mm, vias 0 -> 2
- net N$3: track 0.00 -> 63.5 mm, vias 0 -> 2
- net SCK: track 0.00 -> 60.4 mm, vias 0 -> 4
- net SCL: track 0.00 -> 55.8 mm, vias 0 -> 1
- net N$18: track 0.00 -> 54.5 mm, vias 0 -> 2
- net SDA: track 0.00 -> 53.9 mm, vias 0 -> 1
- net A0: track 0.00 -> 53.1 mm, vias 0 -> 3
- net MOSI: track 0.00 -> 51.6 mm, vias 0 -> 1
- net N$5: track 0.00 -> 49.4 mm, vias 0 -> 2
- net D10: track 0.00 -> 47.7 mm, vias 0 -> 3
- net A1: track 0.00 -> 45.1 mm, vias 0 -> 3
- net 5V_UC: track 0.00 -> 44.6 mm, vias 0 -> 2
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