File: eagle/halloween/halloween2013/connector-amplified/connector-2channel.brd (EAGLE design)
At the start: 30.1 x 18.7 mm, 7 parts, among them J3 RJ12RIGHTANGLE, Q1 BCV27

Commit message: update halloween
Parts:
- added D1, D2: 1N581D1206, lpatiny:LED-1206
Connections:
- net +12V: now also D2.C
- net +5V: now also D1.C
- net N$4: now also D1.A, D2.A
Routing:
- net N$4: track 5.25 -> 13.0 mm
- net +12V: track 44.6 -> 48.5 mm
- net +5V: track 46.5 -> 50.3 mm
Changed lines of the file:
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@@
 <?xml version="1.0" encoding="utf-8"?>
 <!DOCTYPE eagle SYSTEM "eagle.dtd">
-<eagle version="6.4">
+<eagle version="6.1">
 <drawing>
 <settings>
@@
 </class>
 </classes>
-<designrules name="default">
+<designrules>
 <description language="de">&lt;b&gt;EAGLE Design Rules&lt;/b&gt;
 &lt;p&gt;
@@
 <element name="C1" library="resistor" package="C1206" value="0.1uF" x="2.54" y="12.7" rot="MR90"/>
 <element name="C2" library="resistor" package="C1206" value="0.1uF" x="2.54" y="7.62" rot="MR90"/>
+<element name="D1" library="lpatiny" package="LED-1206" value="1N581D1206" x="27.94" y="15.24" rot="MR90"/>
+<element name="D2" library="lpatiny" package="LED-1206" value="1N581D1206" x="27.94" y="12.7" rot="R270"/>
 </elements>
 <signals>
@@
 <wire x1="27.94" y1="2.54" x2="27.94" y2="11.43" width="1.27" layer="16"/>
 <wire x1="27.94" y1="11.43" x2="24.13" y2="11.43" width="1.27" layer="16"/>
+<contactref element="D2" pad="C"/>
+<wire x1="24.384" y1="11.2776" x2="27.8892" y2="11.2776" width="0.4572" layer="1"/>
+<wire x1="24.2316" y1="11.43" x2="24.384" y2="11.2776" width="0.4572" layer="1"/>
+<wire x1="27.8892" y1="11.2776" x2="27.94" y2="11.2" width="0.4572" layer="1"/>
+<wire x1="24.2316" y1="11.43" x2="24.13" y2="11.43" width="0.4572" layer="1"/>
 </signal>
 <signal name="+5V">
@@
 <wire x1="20.32" y1="16.51" x2="20.32" y2="7.62" width="1.27" layer="16"/>
 <wire x1="20.32" y1="7.62" x2="24.13" y2="7.62" width="1.27" layer="16"/>
+<contactref element="D1" pad="C"/>
+<wire x1="24.6888" y1="16.764" x2="27.8892" y2="16.764" width="0.4572" layer="16"/>
+<wire x1="27.8892" y1="16.764" x2="27.94" y2="16.74" width="0.4572" layer="16"/>
+<wire x1="24.6888" y1="16.764" x2="24.13" y2="16.51" width="0.4572" layer="16"/>
 </signal>
 <signal name="N$3">
@@
 <contactref element="Q1" pad="3"/>
 <wire x1="24.13" y1="13.97" x2="18.88" y2="13.97" width="1.27" layer="1"/>
+<contactref element="D1" pad="A"/>
+<contactref element="D2" pad="A"/>
+<wire x1="24.2316" y1="13.8684" x2="27.8892" y2="13.8684" width="0.4572" layer="16"/>
+<wire x1="27.8892" y1="13.8684" x2="27.94" y2="13.74" width="0.4572" layer="16"/>
+<wire x1="24.2316" y1="13.8684" x2="24.13" y2="13.97" width="0.4572" layer="16"/>
+<wire x1="24.6888" y1="14.1732" x2="27.8892" y2="14.1732" width="0.4572" layer="1"/>
+<wire x1="27.8892" y1="14.1732" x2="27.94" y2="14.2" width="0.4572" layer="1"/>
+<wire x1="24.6888" y1="14.1732" x2="24.13" y2="13.97" width="0.4572" layer="1"/>
 </signal>
 </signals>
