File: eagle/halloween/halloween2013/led-driver/led-driver-v1.brd (EAGLE design)
At the start: 48.9 x 49.2 mm, 16 parts, among them IC1 MEGA8-AI, J1 RJ12RIGHTANGLE-I2C, J2 RJ12RIGHTANGLE-I2C

Commit message: Update halloween
Routing:
- net GND: track 2.11 -> 161.3 mm, vias 0 -> 1
- net MISO: track 2.99 -> 109.0 mm, vias 0 -> 1
- net D5: track 0.00 -> 85.1 mm, vias 0 -> 2
- net N$13: track 0.00 -> 77.3 mm, vias 0 -> 1
- net +5V: track 0.00 -> 70.7 mm, vias 0 -> 2
- net RESET: track 1.66 -> 69.4 mm, vias 0 -> 3
- net D4: track 0.00 -> 67.3 mm, vias 0 -> 2
- net MOSI: track 3.89 -> 69.5 mm, vias 0 -> 3
- net D8: track 0.00 -> 62.5 mm, vias 0 -> 2
- net 5V_B: track 0.00 -> 59.0 mm, vias 0 -> 3
- net SCK: track 3.57 -> 59.7 mm, vias 0 -> 2
- net D2: track 0.00 -> 56.1 mm, vias 0 -> 1
- net D9: track 0.00 -> 55.1 mm, vias 0 -> 2
- net D6: track 0.00 -> 49.2 mm, vias 0 -> 3
- net D0: track 0.00 -> 47.6 mm, vias 0 -> 2
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
Commit message: Update 20 leds driver
Parts:
- moved J1 34.3 mm to (6.35, 22.9)
- moved J2 34.3 mm to (43.2, 22.9)
Routing:
- net GND: track 161.3 -> 0.00 mm, vias 1 -> 0
- net MISO: track 109.0 -> 0.00 mm, vias 1 -> 0
- net D5: track 85.1 -> 0.00 mm, vias 2 -> 0
- net N$13: track 77.3 -> 0.00 mm, vias 1 -> 0
- net +5V: track 70.7 -> 0.00 mm, vias 2 -> 0
- net MOSI: track 69.5 -> 0.00 mm, vias 3 -> 0
- net RESET: track 69.4 -> 0.00 mm, vias 3 -> 0
- net D4: track 67.3 -> 0.00 mm, vias 2 -> 0
- net D8: track 62.5 -> 0.00 mm, vias 2 -> 0
- net SCK: track 59.7 -> 0.00 mm, vias 2 -> 0
- net 5V_B: track 59.0 -> 0.00 mm, vias 3 -> 0
- net D2: track 56.1 -> 0.00 mm, vias 1 -> 0
- net D9: track 55.1 -> 0.00 mm, vias 2 -> 0
- net D6: track 49.2 -> 0.00 mm, vias 3 -> 0
- net D0: track 47.6 -> 0.00 mm, vias 2 -> 0
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