File: eagle/modules/femto/v1.1/femto.brd (EAGLE design)
At the start: 50.2 x 25.1 mm, 29 parts, among them IC1 MEGA8-AI, J1 RJ12RIGHTANGLE-I2C, J2 RJ12RIGHTANGLE-I2C

Commit message: Update femto
Routing:
- net GND: track 189.1 -> 118.1 mm, vias 1 -> 0
- net SDA: track 65.3 -> 0.00 mm, vias 3 -> 0
- net SCL: track 58.2 -> 0.00 mm, vias 2 -> 0
- net +5V: track 52.5 -> 0.00 mm, vias 3 -> 0
- net D3: track 43.4 -> 0.00 mm
- net RESET: track 42.5 -> 0.00 mm, vias 2 -> 0
- net MOSI: track 36.1 -> 0.00 mm, vias 2 -> 0
- net MISO: track 30.3 -> 0.00 mm, vias 4 -> 0
- net 5V_B: track 117.7 -> 89.0 mm
- net SCK: track 25.6 -> 0.00 mm, vias 2 -> 0
- net D10: track 23.8 -> 0.13 mm, vias 2 -> 0
- net D9: track 16.9 -> 0.00 mm
- net D6: track 16.6 -> 0.00 mm, vias 1 -> 0
- net N$23: track 14.4 -> 0.00 mm
- net D5: track 13.4 -> 0.00 mm, vias 1 -> 0
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
Commit message: femto routing
Parts:
- removed DB1, DB2, DC1, DC4: (no value), led:LED3MM
- added LED4, LED5, LED6: LED3MM, lpatiny:LED3MM
- added LED7: (no value), adafruit:CHIP-LED0603
- LED3: value (none) -> LED3MM; device adafruit:CHIP-LED0603 -> lpatiny:LED3MM
- moved LED3 14.7 mm to (32.4, 17.8), turned to 90 degrees
- moved LED1 7.62 mm to (18.4, 19.1)
- moved LED2 7.62 mm to (26.0, 19.1)
- renumbered R1 to R8, R2 to R7, RB1 to R5, RB2 to R4, RC1 to R3, RC6 to R6, RD10 to R2C, RD11 to R1A, RD12 to R1B, RD13 to R1C, RD8 to R2A, RD9 to R2B
Connections:
- net GND: now also LED3.K, LED4.K, LED5.K, LED6.K, LED7.C; no longer DB1.K, DB2.K, DC1.K, DC4.K, LED3.C
- net N$1: now also LED2.RED; no longer LED1.RED
- net N$15: now also LED7.A; no longer LED3.A
- net N$16: now also LED3.A; no longer DC1.A
- net N$20: now also LED1.RED; no longer LED2.RED
- net N$21: now also LED1.BLU; no longer LED2.BLU
- net N$22: now also LED1.GRN; no longer LED2.GRN
- net N$23: now also LED6.A; no longer DC4.A
- net N$40: now also LED5.A; no longer DB1.A
- net N$41: now also LED4.A; no longer DB2.A
- net N$7: now also LED2.BLU; no longer LED1.BLU
- net N$8: now also LED2.GRN; no longer LED1.GRN
Routing:
- net GND: track 118.1 -> 189.1 mm, vias 0 -> 1
- net SDA: track 0.00 -> 65.3 mm, vias 0 -> 3
- net SCL: track 0.00 -> 58.2 mm, vias 0 -> 2
- net +5V: track 0.00 -> 52.5 mm, vias 0 -> 3
- net D3: track 0.00 -> 43.4 mm
- net RESET: track 0.00 -> 42.5 mm, vias 0 -> 2
- net MOSI: track 0.00 -> 36.1 mm, vias 0 -> 2
- net MISO: track 0.00 -> 30.3 mm, vias 0 -> 4
- net 5V_B: track 89.0 -> 117.7 mm
- net SCK: track 0.00 -> 25.6 mm, vias 0 -> 2
- net D10: track 0.13 -> 23.8 mm, vias 0 -> 2
- net D9: track 0.00 -> 16.9 mm
- net D6: track 0.00 -> 16.6 mm, vias 0 -> 1
- net N$23: track 0.00 -> 14.4 mm
- net D5: track 0.00 -> 13.4 mm, vias 0 -> 1
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
Commit message: Correct femto
Parts:
- moved J1 3.81 mm to (45.7, 7.62), turned to 90 degrees
- moved C3 3.81 mm to (12.7, 14.6)
- moved J2 3.81 mm to (5.08, 7.62), turned to 270 degrees
- moved C1 3.81 mm to (12.7, 1.91)
- moved C2 3.81 mm to (12.7, 12.1)
Routing:
- net SDA: track 65.3 -> 90.8 mm, vias 3 -> 1
- net GND: track 189.1 -> 164.0 mm
- net D3: track 43.4 -> 18.4 mm, vias 0 -> 2
- net SCL: track 58.2 -> 74.1 mm, vias 2 -> 0
- net N$13: track 58.4 -> 43.8 mm
- net 5V_B: track 117.7 -> 108.0 mm
- net D6: track 16.6 -> 8.46 mm
- net D10: track 23.8 -> 15.7 mm, vias 2 -> 0
- net MISO: track 30.3 -> 22.2 mm, vias 4 -> 2
- net N$23: track 14.4 -> 21.0 mm
- net RESET: track 42.5 -> 36.8 mm, vias 2 -> 3
- net N$41: track 10.2 -> 15.2 mm, vias 0 -> 1
- net +5V: track 52.5 -> 48.0 mm, vias 3 -> 2
- net N$4: track 5.18 -> 9.24 mm, vias 0 -> 2
- net D4: track 12.6 -> 9.25 mm
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
Commit message: Update arduino for soft pwm and 8 mhz
Parts:
- R1A, R2A, R5, R6: value 1k -> 330
- R1B, R1C, R2B, R2C: value 1k -> 229
- R3, R4: value 1k -> 220
Changed lines of the file:
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@@
 <layer number="31" name="tCream" color="7" fill="4" visible="yes" active="yes"/>
 <layer number="32" name="bCream" color="7" fill="5" visible="yes" active="yes"/>
-<layer number="33" name="tFinish" color="6" fill="3" visible="no" active="yes"/>
-<layer number="34" name="bFinish" color="6" fill="6" visible="no" active="yes"/>
+<layer number="33" name="tFinish" color="6" fill="3" visible="yes" active="yes"/>
+<layer number="34" name="bFinish" color="6" fill="6" visible="yes" active="yes"/>
 <layer number="35" name="tGlue" color="7" fill="4" visible="no" active="yes"/>
 <layer number="36" name="bGlue" color="7" fill="5" visible="no" active="yes"/>
@@
 <attribute name="OC_FARNELL" value="9171371" x="3.81" y="3.81" size="1.778" layer="28" rot="MR0" display="off"/>
 </element>
-<element name="R5" library="resistor" package="M1206" value="1k" x="32.385" y="8.89" smashed="yes" rot="MR90">
+<element name="R5" library="resistor" package="M1206" value="330" x="32.385" y="8.89" smashed="yes" rot="MR90">
 <attribute name="VALUE" x="32.0675" y="5.08" size="1.27" layer="28" rot="MR90"/>
 </element>
-<element name="R4" library="resistor" package="M1206" value="1k" x="29.21" y="8.89" smashed="yes" rot="MR90">
+<element name="R4" library="resistor" package="M1206" value="220" x="29.21" y="8.89" smashed="yes" rot="MR90">
 <attribute name="VALUE" x="28.575" y="5.08" size="1.27" layer="28" rot="MR90"/>
 </element>
@@
 <element name="LED2" library="lpatiny" package="LED-TRICOLOR-THROUGHHOLE" value="RGB-COMMON-CATHODE" x="26.035" y="19.05" rot="R270"/>
 <element name="LED1" library="lpatiny" package="LED-TRICOLOR-THROUGHHOLE" value="RGB-COMMON-CATHODE" x="18.415" y="19.05" rot="R270"/>
-<element name="R2A" library="resistor" package="M1206" value="1k" x="31.4325" y="11.43" smashed="yes" rot="R90">
+<element name="R2A" library="resistor" package="M1206" value="330" x="31.4325" y="11.43" smashed="yes" rot="R90">
 <attribute name="VALUE" x="32.0675" y="13.6525" size="1.27" layer="27" rot="R90"/>
 </element>
-<element name="R2B" library="resistor" package="M1206" value="1k" x="25.7175" y="11.43" smashed="yes" rot="R90">
+<element name="R2B" library="resistor" package="M1206" value="229" x="25.7175" y="11.43" smashed="yes" rot="R90">
 <attribute name="VALUE" x="26.3525" y="13.6525" size="1.27" layer="27" rot="R90"/>
 </element>
-<element name="R2C" library="resistor" package="M1206" value="1k" x="28.575" y="11.43" smashed="yes" rot="R90">
+<element name="R2C" library="resistor" package="M1206" value="229" x="28.575" y="11.43" smashed="yes" rot="R90">
 <attribute name="VALUE" x="29.21" y="13.6525" size="1.27" layer="27" rot="R90"/>
 </element>
-<element name="R1A" library="resistor" package="M1206" value="1k" x="22.86" y="11.43" smashed="yes" rot="R90">
+<element name="R1A" library="resistor" package="M1206" value="330" x="22.86" y="11.43" smashed="yes" rot="R90">
 <attribute name="VALUE" x="23.495" y="13.6525" size="1.27" layer="27" rot="R90"/>
 </element>
-<element name="R1B" library="resistor" package="M1206" value="1k" x="17.145" y="11.43" smashed="yes" rot="R90">
+<element name="R1B" library="resistor" package="M1206" value="229" x="17.145" y="11.43" smashed="yes" rot="R90">
 <attribute name="VALUE" x="17.78" y="13.6525" size="1.27" layer="27" rot="R90"/>
 </element>
-<element name="R1C" library="resistor" package="M1206" value="1k" x="20.0025" y="11.43" smashed="yes" rot="R90">
+<element name="R1C" library="resistor" package="M1206" value="229" x="20.0025" y="11.43" smashed="yes" rot="R90">
 <attribute name="VALUE" x="20.6375" y="13.6525" size="1.27" layer="27" rot="R90"/>
 </element>
-<element name="R6" library="resistor" package="M1206" value="1k" x="35.56" y="8.89" smashed="yes" rot="MR90">
+<element name="R6" library="resistor" package="M1206" value="330" x="35.56" y="8.89" smashed="yes" rot="MR90">
 <attribute name="VALUE" x="35.2425" y="5.08" size="1.27" layer="28" rot="MR90"/>
 </element>
@@
 <element name="D1" library="lpatiny" package="LED-1206" value="1N581D1206" x="11.7475" y="20.32" rot="MR270"/>
 <element name="D2" library="lpatiny" package="LED-1206" value="1N581D1206" x="11.7475" y="20.32" rot="R270"/>
-<element name="R3" library="resistor" package="M1206" value="1k" x="34.29" y="11.43" smashed="yes" rot="R90">
+<element name="R3" library="resistor" package="M1206" value="220" x="34.29" y="11.43" smashed="yes" rot="R90">
 <attribute name="VALUE" x="34.925" y="13.6525" size="1.27" layer="27" rot="R90"/>
 </element>
