File: eagle/halloween/halloween2014/Controller/v1.1 - noled/v1.brd (EAGLE design)
At the start: 111.9 x 84.6 mm, 94 parts, among them CON1 SPI, J1 RJ12, J2 RJ12, J3 RJ12, J4 RJ12, J5 RJ12, Q1 BSP75, Q10 BSP75, Q11 BSP75, Q12 BSP75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

Commit message: First proto controller
Parts:
- removed LED13, LED16: GREEN, adafruit:CHIPLED_1206
- removed LED14, LED17: BLUE, adafruit:CHIPLED_1206
- removed LED15, LED3: RED, adafruit:CHIPLED_1206
- removed LED2, LED5, LED6, LED8: Blue, adafruit:CHIPLED_1206
- removed LED7: BLue, adafruit:CHIPLED_1206
- removed R25, R4, R5, R6, R7: 1k, rcl:R0805
- removed RL10, RL11, RL12, RL2, RL8, RL9: 1K, resistor:M0805
- moved X1 202.6 mm to (102.9, 66.0), turned to 270 degrees
- moved R2 180.4 mm to (88.9, 44.5), turned to 90 degrees
- moved R1 174.7 mm to (86.4, 44.5), turned to 90 degrees
- moved U$1 167.5 mm to (92.7, 48.3)
- moved R15 72.7 mm to (24.1, 44.5), flipped to the bottom
- moved C9 72.7 mm to (29.2, 44.5), flipped to the bottom
- moved RESET1 72.7 mm to (26.7, 44.5), flipped to the top
- moved Q11 63.1 mm to (35.6, 35.6)
- moved CON1 37.1 mm to (8.89, 21.6), turned to 270 degrees
- moved Q12 31.4 mm to (43.2, 35.6), turned to 0 degrees
- moved C10 17.3 mm to (30.5, 54.6)
- moved C12 17.3 mm to (33.0, 54.6)
- moved D2 17.3 mm to (25.4, 57.1)
- moved D3 17.3 mm to (25.4, 52.1)
- moved D4 17.3 mm to (25.4, 54.6)
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Connections:
- removed net N$17: LED2.A, R25.1
- removed net N$22: LED6.A, R5.1
- removed net N$30: LED7.A, R6.1
- removed net N$31: LED15.C, RL10.2
- removed net N$33: LED8.A, R7.1
- removed net N$36: LED3.C, RL2.2
- removed net N$37: LED13.C, RL8.2
- removed net N$4: LED5.A, R4.1
- removed net N$40: LED14.C, RL9.2
- removed net N$41: LED16.C, RL11.2
- removed net N$43: LED17.C, RL12.2
- net +5V: no longer LED13.A, LED14.A, LED15.A, LED16.A, LED17.A, LED3.A, R25.2, R4.2, R5.2, R6.2, R7.2
- net N$1: no longer LED6.C
- net N$10: no longer RL11.1
- net N$19: no longer LED8.C
- net N$20: no longer RL10.1
- net N$23: no longer RL12.1
- net N$28: no longer LED5.C
- net N$34: no longer LED2.C
- net N$5: no longer LED7.C
- net N$50: no longer RL8.1
- net N$6: no longer RL9.1
- net N$68: no longer RL2.1
Routing:
- net +5V: track 450.6 -> 406.7 mm
- net GND: track 433.5 -> 474.5 mm
- net N$10: track 0.00 -> 28.0 mm
- net +12V: track 335.7 -> 311.5 mm
- net D8*: track 23.6 -> 0.00 mm
- net A2: track 20.2 -> 0.00 mm
- net N$19: track 24.3 -> 8.97 mm
- net N$34: track 24.3 -> 8.97 mm
- net N$28: track 24.3 -> 8.97 mm
- net N$5: track 24.3 -> 8.97 mm
- net N$1: track 24.3 -> 8.97 mm
- net N$20: track 0.00 -> 15.3 mm
- net N$42: track 0.00 -> 14.6 mm, vias 0 -> 1
- net XTAL1: track 0.00 -> 13.8 mm, vias 0 -> 1
- net N$23: track 0.00 -> 11.5 mm
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Other:
- board size 111.9 x 84.6 mm -> 111.9 x 78.2 mm
