File: eagle/halloween/halloween2014/Controller/v1.1 - noled/v1.sch (EAGLE design)
At the start: 94 parts, among them CON1 SPI, J1 RJ12, J2 RJ12, J3 RJ12, J4 RJ12, J5 RJ12, Q1 BSP75, Q10 BSP75, Q11 BSP75, Q12 BSP75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

Commit message: First proto controller
Parts:
- removed LED13, LED16: GREEN, adafruit:LEDCHIPLED_1206
- removed LED14, LED17: BLUE, adafruit:LEDCHIPLED_1206
- removed LED15, LED3: RED, adafruit:LEDCHIPLED_1206
- removed LED2, LED5, LED6, LED8: Blue, adafruit:LEDCHIPLED_1206
- removed LED7: BLue, adafruit:LEDCHIPLED_1206
- removed R25, R4, R5, R6, R7: 1k, rcl:R-EU_R0805
- removed RL10, RL11, RL12, RL2, RL8, RL9: 1K, resistor:R-EU_M0805
Connections:
- removed net N$17: LED2.A, R25.1
- removed net N$22: LED6.A, R5.1
- removed net N$30: LED7.A, R6.1
- removed net N$31: LED15.C, RL10.2
- removed net N$33: LED8.A, R7.1
- removed net N$36: LED3.C, RL2.2
- removed net N$37: LED13.C, RL8.2
- removed net N$4: LED5.A, R4.1
- removed net N$40: LED14.C, RL9.2
- removed net N$41: LED16.C, RL11.2
- removed net N$43: LED17.C, RL12.2
- net +5V: no longer LED13.A, LED14.A, LED15.A, LED16.A, LED17.A, LED3.A, R25.2, R4.2, R5.2, R6.2, R7.2
- net N$1: no longer LED6.C
- net N$10: no longer RL11.1
- net N$19: no longer LED8.C
- net N$20: no longer RL10.1
- net N$23: no longer RL12.1
- net N$28: no longer LED5.C
- net N$34: no longer LED2.C
- net N$5: no longer LED7.C
- net N$50: no longer RL8.1
- net N$6: no longer RL9.1
- net N$68: no longer RL2.1
