File: eagle/halloween/halloween2014/Controller/v1.1 old bad/v1.sch (EAGLE design)
At the start: 72 parts, among them CON1 SPI, J1 RJ12, J2 RJ12, J3 RJ12, J4 RJ12, J5 RJ12, Q1 BSP75, Q10 BSP75, Q11 BSP75, Q12 BSP75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

Commit message: Update halloween 2014
Connections:
- removed net D14*: Q5.G
- removed net D15*: Q6.G
- net MISO: now also Q5.G
- net RD+: no longer RL7.1
- net RD-: no longer RL1.1
- net RXLED: now also RL1.1
- net SCK: now also Q6.G
- net TXLED: now also RL7.1
Changed lines of the file:
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@@
 </variantdefs>
 <classes>
-<class number="0" name="default" width="0.3048" drill="0">
+<class number="0" name="default" width="0.4064" drill="0">
 </class>
 <class number="1" name="power" width="0.4572" drill="0">
@@
 <class number="2" name="VIN" width="0.4572" drill="0">
 </class>
-<class number="3" name="fine" width="0.3048" drill="0">
+<class number="3" name="fine" width="0.4064" drill="0">
 </class>
-<class number="4" name="aref" width="0.3048" drill="0">
+<class number="4" name="aref" width="0.4064" drill="0">
 </class>
 </classes>
@@
 <pinref part="X1" gate="G$1" pin="1"/>
 <wire x1="-27.94" y1="43.18" x2="-38.1" y2="43.18" width="0.1524" layer="91"/>
+<junction x="-22.86" y="48.26"/>
 </segment>
 <segment>
@@
 <label x="200.66" y="160.02" size="1.778" layer="95"/>
 </segment>
+<segment>
+<pinref part="Q6" gate="G$1" pin="G"/>
+<wire x1="220.98" y1="246.38" x2="215.9" y2="246.38" width="0.1524" layer="91"/>
+<label x="215.9" y="243.84" size="1.778" layer="95"/>
+<junction x="220.98" y="246.38"/>
+</segment>
 </net>
 <net name="MISO" class="0">
@@
 <wire x1="208.28" y1="162.56" x2="200.66" y2="162.56" width="0.1524" layer="91"/>
 <label x="200.66" y="162.56" size="1.778" layer="95"/>
+</segment>
+<segment>
+<pinref part="Q5" gate="G$1" pin="G"/>
+<wire x1="177.8" y1="246.38" x2="172.72" y2="246.38" width="0.1524" layer="91"/>
+<label x="172.72" y="243.84" size="1.778" layer="95"/>
+<junction x="177.8" y="246.38"/>
 </segment>
 </net>
@@
 <net name="RD-" class="0">
 <segment>
-<pinref part="RL1" gate="G$1" pin="1"/>
-<wire x1="-83.82" y1="243.84" x2="-88.9" y2="243.84" width="0.1524" layer="91"/>
-<label x="-93.98" y="243.84" size="1.778" layer="95"/>
-</segment>
-<segment>
 <pinref part="U$4" gate="G$1" pin="D-"/>
 <wire x1="198.12" y1="60.96" x2="180.34" y2="60.96" width="0.1524" layer="91"/>
@@
 </net>
 <net name="RD+" class="0">
-<segment>
-<pinref part="RL7" gate="G$1" pin="1"/>
-<wire x1="-83.82" y1="228.6" x2="-88.9" y2="228.6" width="0.1524" layer="91"/>
-<label x="-93.98" y="228.6" size="1.778" layer="95"/>
-</segment>
 <segment>
 <pinref part="U$4" gate="G$1" pin="D+"/>
@@
 <wire x1="246.38" y1="27.94" x2="261.62" y2="27.94" width="0.1524" layer="91"/>
 <label x="256.54" y="27.94" size="1.778" layer="95"/>
+</segment>
+<segment>
+<pinref part="RL7" gate="G$1" pin="1"/>
+<wire x1="-83.82" y1="228.6" x2="-88.9" y2="228.6" width="0.1524" layer="91"/>
+<label x="-93.98" y="228.6" size="1.778" layer="95"/>
 </segment>
 </net>
@@
 <wire x1="246.38" y1="38.1" x2="261.62" y2="38.1" width="0.1524" layer="91"/>
 <label x="256.54" y="38.1" size="1.778" layer="95"/>
+</segment>
+<segment>
+<pinref part="RL1" gate="G$1" pin="1"/>
+<wire x1="-83.82" y1="243.84" x2="-88.9" y2="243.84" width="0.1524" layer="91"/>
+<label x="-93.98" y="243.84" size="1.778" layer="95"/>
 </segment>
 </net>
@@
 <pinref part="R1" gate="G$1" pin="1"/>
 <wire x1="-25.4" y1="63.5" x2="-27.94" y2="63.5" width="0.1524" layer="91"/>
+<junction x="-15.24" y="60.96"/>
 </segment>
 </net>
@@
 <pinref part="R2" gate="G$1" pin="1"/>
 <wire x1="-15.24" y1="58.42" x2="-27.94" y2="58.42" width="0.1524" layer="91"/>
+<junction x="-15.24" y="58.42"/>
 </segment>
 </net>
@@
 </segment>
 </net>
-<net name="D15*" class="0">
-<segment>
-<pinref part="Q6" gate="G$1" pin="G"/>
-<wire x1="220.98" y1="246.38" x2="215.9" y2="246.38" width="0.1524" layer="91"/>
-<label x="215.9" y="243.84" size="1.778" layer="95"/>
-<junction x="220.98" y="246.38"/>
-</segment>
-</net>
-<net name="D14*" class="0">
-<segment>
-<pinref part="Q5" gate="G$1" pin="G"/>
-<wire x1="177.8" y1="246.38" x2="172.72" y2="246.38" width="0.1524" layer="91"/>
-<label x="172.72" y="243.84" size="1.778" layer="95"/>
-<junction x="177.8" y="246.38"/>
-</segment>
-</net>
 </nets>
 </sheet>
 </sheets>
-<errors>
-</errors>
 </schematic>
 </drawing>
