File: eagle/halloween/halloween2014/Controller/v1.2/v1.sch (EAGLE design)
At the start: 72 parts, among them CON1 SPI, J1 RJ12, J2 RJ12, J3 RJ12, J4 RJ12, J5 RJ12, Q1 BSP75, Q10 BSP75, Q11 BSP75, Q12 BSP75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

Commit message: Update halloween 2014 and seeed proces file
Parts:
- added LED1: RED, adafruit:LEDCHIP-LED0805
- added R4: 1K, rcl:R-EU_R0805
- LED10, LED4: value RED -> GREEN
Connections:
- new net N$4: LED1.A, R4.1
- net D13*: now also R4.2
- net GND: now also LED1.C
Changed lines of the file:
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@@
 <part name="GND25" library="supply1" deviceset="GND" device=""/>
 <part name="U$6" library="lpatiny" deviceset="KPJX-4S-S" device=""/>
-<part name="LED10" library="adafruit" deviceset="LED" device="CHIP-LED0805" value="RED"/>
+<part name="LED10" library="adafruit" deviceset="LED" device="CHIP-LED0805" value="GREEN"/>
 <part name="RL3" library="rcl" deviceset="R-EU_" device="R0805" value="1K"/>
 <part name="F2" library="lpatiny" deviceset="POLYSWITCH" device="SMD1812" value="1.2A"/>
@@
 <part name="D2" library="lpatiny" deviceset="1N581*" device="D1206" value="1N581D1206"/>
 <part name="GND15" library="supply1" deviceset="GND" device=""/>
-<part name="LED4" library="adafruit" deviceset="LED" device="CHIP-LED0805" value="RED"/>
+<part name="LED4" library="adafruit" deviceset="LED" device="CHIP-LED0805" value="GREEN"/>
 <part name="RL4" library="resistor" deviceset="R-EU_" device="R0805" value="1K"/>
 <part name="D3" library="lpatiny" deviceset="1N581*" device="D1206" value="1N581D1206"/>
@@
 <part name="GND19" library="supply1" deviceset="GND" device=""/>
 <part name="X1" library="con-lumberg" deviceset="1503_09" device=""/>
+<part name="LED1" library="adafruit" deviceset="LED" device="CHIP-LED0805" value="RED"/>
+<part name="R4" library="rcl" deviceset="R-EU_" device="R0805" value="1K"/>
+<part name="GND20" library="supply1" deviceset="GND" device=""/>
 </parts>
 <sheets>
@@
 <instance part="U$8" gate="G$1" x="177.8" y="86.36"/>
 <instance part="R3" gate="G$1" x="266.7" y="71.12" rot="R180"/>
-<instance part="GND4" gate="1" x="279.4" y="66.04"/>
+<instance part="GND4" gate="1" x="279.4" y="68.58"/>
 <instance part="R15" gate="G$1" x="137.16" y="101.6" rot="R90"/>
 <instance part="C3" gate="G$1" x="144.78" y="53.34" rot="R90"/>
@@
 <instance part="GND19" gate="1" x="17.78" y="45.72"/>
 <instance part="X1" gate="G$1" x="-43.18" y="48.26" rot="MR0"/>
+<instance part="LED1" gate="G$1" x="276.86" y="60.96" rot="MR270"/>
+<instance part="R4" gate="G$1" x="266.7" y="60.96" rot="MR0"/>
+<instance part="GND20" gate="1" x="287.02" y="58.42"/>
 </instances>
 <busses>
@@
 <pinref part="GND4" gate="1" pin="GND"/>
 <wire x1="271.78" y1="71.12" x2="279.4" y2="71.12" width="0.1524" layer="91"/>
-<wire x1="279.4" y1="71.12" x2="279.4" y2="68.58" width="0.1524" layer="91"/>
 </segment>
 <segment>
@@
 <wire x1="10.16" y1="48.26" x2="17.78" y2="48.26" width="0.1524" layer="91"/>
 <pinref part="GND19" gate="1" pin="GND"/>
+</segment>
+<segment>
+<pinref part="LED1" gate="G$1" pin="C"/>
+<wire x1="281.94" y1="60.96" x2="287.02" y2="60.96" width="0.1524" layer="91"/>
+<pinref part="GND20" gate="1" pin="GND"/>
 </segment>
 </net>
@@
 <wire x1="246.38" y1="60.96" x2="261.62" y2="60.96" width="0.1524" layer="91"/>
 <label x="256.54" y="60.96" size="1.778" layer="95"/>
+<pinref part="R4" gate="G$1" pin="2"/>
 </segment>
 </net>
@@
 </segment>
 </net>
+<net name="N$4" class="0">
+<segment>
+<wire x1="271.78" y1="60.96" x2="274.32" y2="60.96" width="0.1524" layer="91"/>
+<pinref part="R4" gate="G$1" pin="1"/>
+<pinref part="LED1" gate="G$1" pin="A"/>
+</segment>
+</net>

Commit message: Update halloween, corredt D8 - D10
Connections:
- net D10*: now also Q2.G
- net D8*: no longer Q2.G
Changed lines of the file:
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@@
 <?xml version="1.0" encoding="utf-8"?>
 <!DOCTYPE eagle SYSTEM "eagle.dtd">
-<eagle version="6.5.0">
+<eagle version="7.1.0">
 <drawing>
 <settings>
@@
 <label x="256.54" y="53.34" size="1.778" layer="95"/>
 </segment>
+<segment>
+<pinref part="Q2" gate="G$1" pin="G"/>
+<wire x1="91.44" y1="246.38" x2="86.36" y2="246.38" width="0.1524" layer="91"/>
+<label x="86.36" y="243.84" size="1.778" layer="95"/>
+</segment>
 </net>
 <net name="HWB" class="0">
@@
 </segment>
 <segment>
-<pinref part="Q2" gate="G$1" pin="G"/>
-<wire x1="91.44" y1="246.38" x2="86.36" y2="246.38" width="0.1524" layer="91"/>
-<label x="86.36" y="243.84" size="1.778" layer="95"/>
-</segment>
-<segment>
