File: eagle/spectrophotometer/v1.0/femto.brd (EAGLE design)
At the start: 50.2 x 25.1 mm, 29 parts, among them IC1 MEGA8-AI, J1 RJ12RIGHTANGLE-I2C, J2 RJ12RIGHTANGLE-I2C

Commit message: Update femto
Parts:
- removed C1, C2: 0.1uF, resistor:C1206
- removed C3: 10uF, resistor:C1206
- removed CON2: (no value), lpatiny:TC2030-MCP
- removed D1, D2: 1N581D1206, lpatiny:LED-1206
- removed IC1: MEGA8-AI, atmel:TQFP32-08
- removed J1, J2: RJ12RIGHTANGLE-I2C, lpatiny:RJ12-RIGHTANGLE-I2C
- removed JP1: (no value), SparkFun:SCREWTERMINAL-3.5MM-2
- removed LED5, LED6: LED3MM, lpatiny:LED3MM
- removed LED7: (no value), adafruit:CHIP-LED0603
- removed R1A, R1B, R1C, R2A, R2B, R2C, R5, R6: 1k, resistor:M1206
- removed R7: 10k, SparkFun:0603-RES
- removed R8: 10k, resistor:M1206
- added CON1: CONN:LEDS, lpatiny:IDC-2*3
- added R1, R2: 1K, rcl:R0805
- LED1, LED2: value RGB-COMMON-CATHODE -> RED; device lpatiny:LED-TRICOLOR-THROUGHHOLE -> adafruit:CHIP-LED0805
- LED3, LED4: value LED3MM -> RED; device lpatiny:LED3MM -> adafruit:CHIP-LED0805
- R3, R4: value 1k -> 1K; device resistor:M1206 -> rcl:R0805
- moved LED1 50.7 mm to (54.6, 54.6), turned to 0 degrees
- moved LED2 26.8 mm to (41.9, 40.6), turned to 0 degrees
- moved R3 15.5 mm to (47.0, 20.3), turned to 0 degrees
- moved LED3 13.0 mm to (41.9, 26.7), turned to 0 degrees
- moved R4 12.0 mm to (40.6, 12.7), flipped to the top, turned to 0 degrees
- moved LED4 5.24 mm to (41.9, 19.1), turned to 0 degrees
Connections:
- removed net +5V: C1.1, C2.1, C3.1, D1.C, D2.C, IC1.18, IC1.4, IC1.6, R7.1, R8.2
- removed net 5V_A: CON2.5V, D1.A
- removed net 5V_B: D2.A, J1.+5V, J2.+5V, JP1.1
- removed net A0: IC1.23
- removed net A1: IC1.24
- removed net A2: IC1.25
- removed net A3: IC1.26
- removed net A6: IC1.19
- removed net A7: IC1.22
- removed net B0: IC1.12, R1C.1
- removed net D10: IC1.14, R4.1
- removed net D2: IC1.32
- removed net D3: IC1.1, R6.1
- removed net D4: IC1.2, R3.1
- removed net D5: IC1.9, R2A.1
- removed net D6: IC1.10, R2C.1
- removed net D7: IC1.11, R1A.1
- removed net D9: IC1.13, R5.1
- removed net MISO: CON2.MISO, IC1.16
- removed net MOSI: CON2.MOSI, IC1.15, R2B.1
- removed net N$13: J1.+12V, J2.+12V
- removed net N$15: LED7.A, R7.2
- removed net N$16: LED3.A, R3.2
- removed net N$20: LED1.RED, R1A.2
- removed net N$21: LED1.BLU, R1B.2
- removed net N$22: LED1.GRN, R1C.2
- removed net N$23: LED6.A, R6.2
- removed net N$40: LED5.A, R5.2
- removed net N$41: LED4.A, R4.2
- removed net N$7: LED2.BLU, R2B.2
- removed net N$8: LED2.GRN, R2C.2
- removed net RESET: CON2.RESET, IC1.29, R8.1
- removed net RX: IC1.30
- removed net SCK: CON2.SCK, IC1.17, R1B.1
- removed net SCL: IC1.28, J1.SCL, J2.SCL
- removed net SDA: IC1.27, J1.SDA, J2.SDA
- removed net TX: IC1.31
- new net D13*: R1.2
- new net D13*1: R2.2
- new net D13*2: R3.2
- new net D13*3: R4.2
- new net N$2: LED2.A, R2.1
- new net N$3: LED3.A, R3.1
- net GND: now also LED1.C, LED2.C, LED3.C, LED4.C; no longer C2.2, C3.2, CON2.GND, IC1.21, IC1.3, IC1.5, J1.GND1, J1.GND2, J2.GND1, J2.GND2, JP1.2, LED1.GND, LED2.GND, LED3.K, LED4.K, LED5.K, LED6.K, LED7.C
- net N$1: now also LED1.A, R1.1; no longer LED2.RED, R2A.2
- net N$4: now also LED4.A, R4.1; no longer C1.2, IC1.20
Routing:
- net 5V_B: track 105.7 -> 0.00 mm
- net GND: track 102.2 -> 0.00 mm
- net N$13: track 43.8 -> 0.00 mm
- net RESET: track 4.94 -> 0.00 mm
