File: eagle/spectrophotometer/v1.0/femto.sch (EAGLE design)
At the start: 29 parts, among them IC1 MEGA8-AI, J1 RJ12RIGHTANGLE-I2C, J2 RJ12RIGHTANGLE-I2C

Commit message: Update femto
Parts:
- removed C1, C2: 0.1uF, resistor:C-EUC1206
- removed C3: 10uF, resistor:C-EUC1206
- removed CON2: (no value), lpatiny:TINYISPTAG
- removed D1, D2: 1N581D1206, lpatiny:1N581D1206
- removed IC1: MEGA8-AI, atmel:MEGA8-AI
- removed J1, J2: RJ12RIGHTANGLE-I2C, lpatiny:RJ12RIGHTANGLE-I2C
- removed JP1: (no value), SparkFun:M023.5MM
- removed LED5, LED6: LED3MM, lpatiny:LED3MM
- removed LED7: (no value), adafruit:LEDCHIP-LED0603
- removed R1A, R1B, R1C, R2A, R2B, R2C, R5, R6: 1k, resistor:R-EU_M1206
- removed R7: 10k, SparkFun:RESISTOR0603-RES
- removed R8: 10k, resistor:R-EU_M1206
- added CON1: CONN:LEDS, lpatiny:CONN:LEDS
- added R1, R2: 1K, rcl:R-EU_R0805
- LED1, LED2: value RGB-COMMON-CATHODE -> RED; device lpatiny:RGB-COMMON-CATHODE -> adafruit:LEDCHIP-LED0805
- LED3, LED4: value LED3MM -> RED; device lpatiny:LED3MM -> adafruit:LEDCHIP-LED0805
- R3, R4: value 1k -> 1K; device resistor:R-EU_M1206 -> rcl:R-EU_R0805
Connections:
- removed net +5V: C1.1, C2.1, C3.1, D1.C, D2.C, IC1.AVCC, IC1.VCC@1, IC1.VCC@2, R7.1, R8.2
- removed net 5V_A: CON2.VCC, D1.A
- removed net 5V_B: D2.A, J1.5, J2.5, JP1.1
- removed net A0: IC1.PC0(ADC0)
- removed net A1: IC1.PC1(ADC1)
- removed net A2: IC1.PC2(ADC2)
- removed net A3: IC1.PC3(ADC3)
- removed net A6: IC1.ADC6
- removed net A7: IC1.ADC7
- removed net B0: IC1.PB0(ICP), R1C.1
- removed net D10: IC1.PB2(SS/OC1B), R4.1
- removed net D2: IC1.PD2(INT0)
- removed net D3: IC1.PD3(INT1), R6.1
- removed net D4: IC1.PD4(XCK/T0), R3.1
- removed net D5: IC1.PD5(T1), R2A.1
- removed net D6: IC1.PD6(AIN0), R2C.1
- removed net D7: IC1.PD7(AIN1), R1A.1
- removed net D9: IC1.PB1(OC1A), R5.1
- removed net MISO: CON2.MISO, IC1.PB4(MISO)
- removed net MOSI: CON2.MOSI, IC1.PB3(MOSI/OC2), R2B.1
- removed net N$13: J1.1, J2.1
- removed net N$15: LED7.A, R7.2
- removed net N$16: LED3.A, R3.2
- removed net N$20: LED1.CRED, R1A.2
- removed net N$21: LED1.CBLUE, R1B.2
- removed net N$22: LED1.CGREEN, R1C.2
- removed net N$23: LED6.A, R6.2
- removed net N$40: LED5.A, R5.2
- removed net N$41: LED4.A, R4.2
- removed net N$7: LED2.CBLUE, R2B.2
- removed net N$8: LED2.CGREEN, R2C.2
- removed net RESET: CON2.RESET, IC1.PC6(/RESET), R8.1
- removed net RX: IC1.PD0(RXD)
- removed net SCK: CON2.SCK, IC1.PB5(SCK), R1B.1
- removed net SCL: IC1.PC5(ADC5/SCL), J1.2, J2.2
- removed net SDA: IC1.PC4(ADC4/SDA), J1.3, J2.3
- removed net TX: IC1.PD1(TXD)
- new net D13*: R1.2
- new net D13*1: R2.2
- new net D13*2: R3.2
- new net D13*3: R4.2
- new net N$2: LED2.A, R2.1
- new net N$3: LED3.A, R3.1
- net GND: now also LED1.C, LED2.C; no longer C2.2, C3.2, CON2.GND, IC1.GND, IC1.GND@1, IC1.GND@2, J1.4, J1.6, J2.4, J2.6, JP1.2, LED1.A2, LED2.A2, LED5.C, LED6.C, LED7.C
- net N$1: now also LED1.A, R1.1; no longer LED2.CRED, R2A.2
- net N$4: now also LED4.A, R4.1; no longer C1.2, IC1.AREF
Other:
- moved on the sheet: LED3, LED4, R3, R4
