File: eagle/halloween/halloween2015/RGB-driver V1 no routing/RGB-driver-v1.sch (EAGLE design)
At the start: 37 parts, among them IC1 MEGA8-AI, J1 RJ12RIGHTANGLE-I2C, J2 RJ12RIGHTANGLE-I2C, Q1 BSP75, Q10 BSP75, Q11 BSP75, Q12 BSP75, Q13 BSP75, Q14 BSP75, Q15 BSP75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

Commit message: Update libraries
t st# Please enter the commit message for your changes. Lines starting
Connections:
- net N$22 renamed GND
- net N$25 renamed +5V_HP
Changed lines of the file:
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@@
 <part name="RGB-J1" library="lpatiny" deviceset="RJ12" device="STRAIGHT-RGB" value="RJ12"/>
 <part name="GND5" library="supply1" deviceset="GND" device=""/>
-<part name="P+41" library="supply2" deviceset="+5V" device=""/>
+<part name="P+41" library="supply2" deviceset="+5V/2" device=""/>
 <part name="P+42" library="supply2" deviceset="+12V" device=""/>
 <part name="Q8" library="infineon" deviceset="BSP613P" device="" value="BSP75"/>
@@
 <part name="RGB-J2" library="lpatiny" deviceset="RJ12" device="STRAIGHT-RGB" value="RJ12"/>
 <part name="GND3" library="supply1" deviceset="GND" device=""/>
-<part name="P+1" library="supply2" deviceset="+5V" device=""/>
+<part name="P+1" library="supply2" deviceset="+5V/2" device=""/>
 <part name="P+4" library="supply2" deviceset="+12V" device=""/>
 <part name="Q7" library="infineon" deviceset="BSP613P" device="" value="BSP75"/>
@@
 <part name="RGB-J3" library="lpatiny" deviceset="RJ12" device="STRAIGHT-RGB" value="RJ12"/>
 <part name="GND11" library="supply1" deviceset="GND" device=""/>
-<part name="P+7" library="supply2" deviceset="+5V" device=""/>
+<part name="P+7" library="supply2" deviceset="+5V/2" device=""/>
 <part name="P+8" library="supply2" deviceset="+12V" device=""/>
 <part name="Q1" library="infineon" deviceset="BSP613P" device="" value="BSP75"/>
@@
 <part name="RGB-J4" library="lpatiny" deviceset="RJ12" device="STRAIGHT-RGB" value="RJ12"/>
 <part name="GND15" library="supply1" deviceset="GND" device=""/>
-<part name="P+9" library="supply2" deviceset="+5V" device=""/>
+<part name="P+9" library="supply2" deviceset="+5V/2" device=""/>
 <part name="P+10" library="supply2" deviceset="+12V" device=""/>
 <part name="Q4" library="infineon" deviceset="BSP613P" device="" value="BSP75"/>
@@
 <part name="RGB-J5" library="lpatiny" deviceset="RJ12" device="STRAIGHT-RGB" value="RJ12"/>
 <part name="GND19" library="supply1" deviceset="GND" device=""/>
-<part name="P+11" library="supply2" deviceset="+5V" device=""/>
+<part name="P+11" library="supply2" deviceset="+5V/2" device=""/>
 <part name="P+12" library="supply2" deviceset="+12V" device=""/>
 <part name="Q13" library="infineon" deviceset="BSP613P" device="" value="BSP75"/>
@@
 <part name="RGB-J6" library="lpatiny" deviceset="RJ12" device="STRAIGHT-RGB" value="RJ12"/>
 <part name="GND23" library="supply1" deviceset="GND" device=""/>
-<part name="P+13" library="supply2" deviceset="+5V" device=""/>
+<part name="P+13" library="supply2" deviceset="+5V/2" device=""/>
 <part name="P+14" library="supply2" deviceset="+12V" device=""/>
 <part name="Q16" library="infineon" deviceset="BSP613P" device="" value="BSP75"/>
@@
 <part name="GND27" library="supply1" deviceset="GND" device=""/>
 <part name="SUPPLY1" library="supply2" deviceset="+12V" device=""/>
-<part name="SUPPLY2" library="supply2" deviceset="+5V" device=""/>
+<part name="SUPPLY2" library="supply2" deviceset="+5V/2" device=""/>
 </parts>
 <sheets>
@@
 <attribute name="VALUE" x="154.305" y="94.615" size="1.27" layer="96" rot="R90"/>
 </instance>
-<instance part="P+41" gate="+5V" x="149.86" y="93.98" smashed="yes" rot="R270">
+<instance part="P+41" gate="G$1" x="149.86" y="93.98" smashed="yes" rot="R270">
 <attribute name="VALUE" x="150.495" y="94.615" size="1.27" layer="96" rot="R90"/>
 </instance>
@@
 <attribute name="VALUE" x="210.185" y="94.615" size="1.27" layer="96" rot="R90"/>
 </instance>
-<instance part="P+1" gate="+5V" x="205.74" y="93.98" smashed="yes" rot="R270">
+<instance part="P+1" gate="G$1" x="205.74" y="93.98" smashed="yes" rot="R270">
 <attribute name="VALUE" x="206.375" y="94.615" size="1.27" layer="96" rot="R90"/>
 </instance>
@@
 <attribute name="VALUE" x="154.305" y="46.355" size="1.27" layer="96" rot="R90"/>
 </instance>
-<instance part="P+7" gate="+5V" x="149.86" y="45.72" smashed="yes" rot="R270">
+<instance part="P+7" gate="G$1" x="149.86" y="45.72" smashed="yes" rot="R270">
 <attribute name="VALUE" x="150.495" y="46.355" size="1.27" layer="96" rot="R90"/>
 </instance>
@@
 <attribute name="VALUE" x="210.185" y="46.355" size="1.27" layer="96" rot="R90"/>
 </instance>
-<instance part="P+9" gate="+5V" x="205.74" y="45.72" smashed="yes" rot="R270">
+<instance part="P+9" gate="G$1" x="205.74" y="45.72" smashed="yes" rot="R270">
 <attribute name="VALUE" x="206.375" y="46.355" size="1.27" layer="96" rot="R90"/>
 </instance>
@@
 <attribute name="VALUE" x="154.305" y="0.635" size="1.27" layer="96" rot="R90"/>
 </instance>
-<instance part="P+11" gate="+5V" x="149.86" y="0" smashed="yes" rot="R270">
+<instance part="P+11" gate="G$1" x="149.86" y="0" smashed="yes" rot="R270">
 <attribute name="VALUE" x="150.495" y="0.635" size="1.27" layer="96" rot="R90"/>
 </instance>
@@
 <attribute name="VALUE" x="210.185" y="0.635" size="1.27" layer="96" rot="R90"/>
 </instance>
-<instance part="P+13" gate="+5V" x="205.74" y="0" smashed="yes" rot="R270">
+<instance part="P+13" gate="G$1" x="205.74" y="0" smashed="yes" rot="R270">
 <attribute name="VALUE" x="206.375" y="0.635" size="1.27" layer="96" rot="R90"/>
 </instance>
@@
 <instance part="GND27" gate="1" x="86.36" y="-30.48"/>
 <instance part="SUPPLY1" gate="+12V" x="99.06" y="-20.32"/>
-<instance part="SUPPLY2" gate="+5V" x="99.06" y="-33.02" rot="R180"/>
+<instance part="SUPPLY2" gate="G$1" x="99.06" y="-33.02" rot="R180"/>
 </instances>
 <busses>
 </busses>
 <nets>
-<net name="N$22" class="1">
+<net name="GND" class="1">
 <segment>
 <pinref part="IC1" gate="G$1" pin="GND@2"/>
@@
 <wire x1="86.36" y1="-27.94" x2="106.68" y2="-27.94" width="0.1524" layer="91"/>
 <wire x1="106.68" y1="-27.94" x2="106.68" y2="-25.4" width="0.1524" layer="91"/>
+<junction x="106.68" y="-27.94"/>
 </segment>
 </net>
@@
 <pinref part="R8" gate="G$1" pin="1"/>
 <wire x1="33.02" y1="68.58" x2="35.56" y2="68.58" width="0.1524" layer="91"/>
+<label x="32.004" y="69.088" size="0.8128" layer="95"/>
 </segment>
 <segment>
@@
 </segment>
 </net>
-<net name="N$10" class="4">
-<segment>
-<pinref part="RGB-J2" gate="G$1" pin="3"/>
-<pinref part="Q11" gate="G$1" pin="D@1"/>
-<wire x1="198.12" y1="99.06" x2="198.12" y2="88.9" width="0.1524" layer="91"/>
-<junction x="198.12" y="88.9"/>
-</segment>
-</net>
 <net name="N$20" class="4">
 <segment>
@@
 </segment>
 </net>
-<net name="N$1" class="4">
-<segment>
-<pinref part="RGB-J3" gate="G$1" pin="3"/>
-<pinref part="Q2" gate="G$1" pin="D@1"/>
-<wire x1="142.24" y1="50.8" x2="142.24" y2="40.64" width="0.1524" layer="91"/>
-<junction x="142.24" y="40.64"/>
-</segment>
-</net>
 <net name="N$2" class="4">
 <segment>
@@
 </segment>
 </net>
-<net name="N$25" class="1">
+<net name="+5V_HP" class="1">
 <segment>
 <pinref part="J3" gate="G$1" pin="4"/>
 <wire x1="106.68" y1="-30.48" x2="99.06" y2="-30.48" width="0.1524" layer="91"/>
-<pinref part="SUPPLY2" gate="+5V" pin="+5V"/>
+<pinref part="SUPPLY2" gate="G$1" pin="+5V/2"/>
+<label x="101.346" y="-32.004" size="0.8128" layer="95"/>
 </segment>
 <segment>
 <wire x1="147.32" y1="0" x2="147.32" y2="5.08" width="0.1524" layer="91"/>
 <pinref part="RGB-J5" gate="G$1" pin="5"/>
-<pinref part="P+11" gate="+5V" pin="+5V"/>
+<pinref part="P+11" gate="G$1" pin="+5V/2"/>
+<label x="146.05" y="2.032" size="0.8128" layer="95" rot="R270"/>
 </segment>
 <segment>
 <wire x1="203.2" y1="0" x2="203.2" y2="5.08" width="0.1524" layer="91"/>
 <pinref part="RGB-J6" gate="G$1" pin="5"/>
-<pinref part="P+13" gate="+5V" pin="+5V"/>
+<pinref part="P+13" gate="G$1" pin="+5V/2"/>
+<label x="202.184" y="2.032" size="0.8128" layer="95" rot="R270"/>
 </segment>
 <segment>
 <wire x1="147.32" y1="45.72" x2="147.32" y2="50.8" width="0.1524" layer="91"/>
 <pinref part="RGB-J3" gate="G$1" pin="5"/>
-<pinref part="P+7" gate="+5V" pin="+5V"/>
+<pinref part="P+7" gate="G$1" pin="+5V/2"/>
+<label x="145.796" y="48.006" size="0.8128" layer="95" rot="R270"/>
 </segment>
 <segment>
 <wire x1="203.2" y1="45.72" x2="203.2" y2="50.8" width="0.1524" layer="91"/>
 <pinref part="RGB-J4" gate="G$1" pin="5"/>
-<pinref part="P+9" gate="+5V" pin="+5V"/>
+<pinref part="P+9" gate="G$1" pin="+5V/2"/>
+<label x="201.676" y="48.006" size="0.8128" layer="95" rot="R270"/>
 </segment>
 <segment>
 <wire x1="203.2" y1="93.98" x2="203.2" y2="99.06" width="0.1524" layer="91"/>
 <pinref part="RGB-J2" gate="G$1" pin="5"/>
-<pinref part="P+1" gate="+5V" pin="+5V"/>
+<pinref part="P+1" gate="G$1" pin="+5V/2"/>
+<label x="201.93" y="96.774" size="0.8128" layer="95" rot="R270"/>
 </segment>
 <segment>
 <wire x1="147.32" y1="93.98" x2="147.32" y2="99.06" width="0.1524" layer="91"/>
 <pinref part="RGB-J1" gate="G$1" pin="5"/>
-<pinref part="P+41" gate="+5V" pin="+5V"/>
+<pinref part="P+41" gate="G$1" pin="+5V/2"/>
+<label x="145.796" y="96.266" size="0.8128" layer="95" rot="R270"/>
+</segment>
+</net>
+<net name="N$10" class="0">
+<segment>
+<pinref part="RGB-J2" gate="G$1" pin="3"/>
+<pinref part="Q11" gate="G$1" pin="D@1"/>
+<wire x1="198.12" y1="99.06" x2="198.12" y2="88.9" width="0.1524" layer="91"/>
+<junction x="198.12" y="88.9"/>
+</segment>
+</net>
+<net name="N$1" class="0">
+<segment>
+<pinref part="RGB-J3" gate="G$1" pin="3"/>
+<pinref part="Q2" gate="G$1" pin="D@1"/>
+<wire x1="142.24" y1="50.8" x2="142.24" y2="40.64" width="0.1524" layer="91"/>
+<junction x="142.24" y="40.64"/>
 </segment>
 </net>
@@
 </sheet>
 </sheets>
+<errors>
+</errors>
 </schematic>
 </drawing>
